File: Installation-01.sch (KiCad schematic (older format))
At the start: 382 parts, among them J2 Conn_ARM_JTAG_SWD_10, U1 STM32F072CBTx, U2 MCP1700-3302E_SOT23, U2 USBLC6-2SC6

Commit message: added usb hub back into keyboard
Parts:
- added C? (x19): 0.1u, symbol Device:C_Small
- added C? (x2): 10u, symbol Device:C_Small
- added C? (x2): 100n, symbol Device:C_Small
- added C? (x3): 4.7n, symbol Device:C_Small
- added C? (x2): 10p, symbol Device:C_Small
- added C? (x4): 150u, symbol Device:C_Small
- added D?: 1N914, Diode_THT:D_DO-35_SOD27_P7.62mm_Horizontal, symbol Diode:1N914
- added JOUT1, JOUT2, JOUT3: USB_C_Receptacle_USB2.0, symbol Connector:USB_C_Receptacle_USB2.0
- added KEEBSWITCH1, OUTSWITCH1, OUTSWITCH2, OUTSWITCH3: TPS2001CDGNR, DGN8_1P89X1P57, symbol TPS2001CDGNR:TPS2001CDGNR
- added R?: 9.53k, symbol Device:R_Small
- added R? (x5): 10k, symbol Device:R_Small
- added R?: 90.9k, symbol Device:R_Small
- added R?: 10M, symbol Device:R_Small
- added R? (x6): 5.1k, symbol Device:R_Small
- added R? (x3): 22k, symbol Device:R_Small
- added U?: TUSB4041I, Package_QFP:HTQFP-64-1EP_10x10mm_P0.5mm_EP8x8mm_Mask4.4x4.4mm_ThermalVias, symbol Interface_USB:TUSB4041I
- added U?: MCP1700-1202E_SOT23, Package_TO_SOT_SMD:SOT-23, symbol Regulator_Linear:MCP1700-1202E_SOT23
- added Y?: 24MHz, symbol Device:Crystal
Connections:
- net labels added: 1.2V, DOUT1+, DOUT1-, DOUT2+, DOUT2-, DOUT3+, DOUT3-, Keeb_D+, Keeb_D-, OUT1VBUS, OUT2VBUS, OUT3VBUS, OVERCUR1, OVERCUR2, OVERCUR3, OVERCUR4, PWRCTL1, PWRCTL2, PWRCTL3, PWRCTL4, VDD33_USB, VDD_USB
- wire segments 867 -> 1159
- no-connect marks 5 -> 20
Other:
- moved on the sheet: C1, C10, C11, C12, C2, C3, C4, C5, C6, C7, C8, C9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

Commit message: Add hotswap sockets
Parts:
- removed D?: D, symbol Device:D
- removed MX?: Lead, symbol MX_Alps_Hybrid:MX-NoLED
- added C143, C144: 100n, CP_EIA_2012_15_AVX-P, symbol Device:C_Small
- added D5: B260, Diode_SMD:D_SMB, symbol Diode:B260
- added D6: 1N914, Diode_THT:D_DO-35_SOD27_P7.62mm_Horizontal, symbol Diode:1N914
- added F2: Polyfuse_Small, Fuse_1206_3216Metric, symbol Device:Polyfuse_Small
- added U5: MCP1700-3302E_SOT23, Package_TO_SOT_SMD:SOT-23, symbol Regulator_Linear:MCP1700-3302E_SOT23
- C1, C10, C11, C12, C2, C3, C4, C5, C6, C7, C8, C9: footprint (none) -> CP_EIA_2012_15_AVX-P
- C100, C101, C102, C103, C104, C105, C106, C107, C108, C109, C110, C111, C112, C113, C114, C115, C116, C117, C118, C119, C120, C121, C122, C123, C124, C125, C126, C127, C128, C129, C13, C130, C131, C132, C133, C134, C135, C136, C137, C138, C139, C14, C140, C141, C142, C145, C15, C16, C17, C18, C19, C20, C21, C22, C23, C24, C25, C26, C27, C28, C29, C30, C31, C32, C33, C34, C35, C36, C37, C38, C39, C40, C41, C42, C43, C44, C45, C46, C47, C48, C49, C50, C51, C52, C53, C54, C55, C56, C57, C58, C59, C60, C61, C62, C63, C64, C65, C66, C67, C68, C69, C70, C71, C72, C73, C74, C75, C76, C77, C78, C79, C80, C81, C82, C83, C84, C85, C86, C87, C88, C89, C90, C91, C92, C93, C94, C95, C96, C97, C98, C99: renamed from C?; footprint (none) -> CP_EIA_2012_15_AVX-P
- D10, D11, D12, D13, D14, D15, D16, D17, D18, D19, D20, D21, D22, D23, D24, D25, D26, D27, D28, D29, D30, D31, D32, D33, D34, D35, D37, D38, D39, D40, D41, D42, D43, D44, D45, D46, D47, D48, D49, D50, D51, D52, D53, D54, D55, D56, D57, D58, D59, D60, D61, D62, D63, D64, D65, D66, D67, D68, D69, D7, D70, D71, D72, D73, D74, D75, D76, D77, D78, D79, D8, D80, D81, D82, D83, D84, D85, D86, D87, D88, D9: renamed from D?; footprint (none) -> D_SOD_123
- F1: footprint (none) -> Fuse_1206_3216Metric
- JIN1, JOUT1, JOUT2, JOUT3: footprint (none) -> Type-C:USB_C_GCT_USB4085
- LED1, LED10, LED11, LED12, LED13, LED14, LED15, LED16, LED17, LED18, LED19, LED2, LED20, LED21, LED22, LED23, LED24, LED25, LED26, LED27, LED28, LED29, LED3, LED30, LED31, LED32, LED33, LED34, LED35, LED36, LED37, LED38, LED39, LED4, LED40, LED41, LED42, LED43, LED44, LED45, LED46, LED47, LED48, LED49, LED5, LED50, LED51, LED52, LED53, LED54, LED55, LED56, LED57, LED58, LED59, LED6, LED60, LED61, LED62, LED63, LED64, LED65, LED66, LED67, LED68, LED69, LED7, LED70, LED71, LED72, LED73, LED74, LED75, LED76, LED77, LED78, LED79, LED8, LED80, LED81, LED82, LED9: renamed from LED?; footprint (none) -> WS2812B
- MX1, MX10, MX11, MX13, MX14, MX15, MX16, MX17, MX18, MX19, MX2, MX20, MX21, MX22, MX23, MX25, MX26, MX27, MX28, MX29, MX31, MX32, MX33, MX34, MX35, MX37, MX38, MX39, MX40, MX41, MX43, MX44, MX45, MX46, MX47, MX48, MX49, MX50, MX51, MX52, MX53, MX55, MX56, MX57, MX58, MX59, MX6, MX60, MX61, MX62, MX63, MX64, MX65, MX66, MX67, MX68, MX69, MX7, MX70, MX72, MX73, MX74, MX75, MX77, MX78, MX8, MX81, MX82, MX9: renamed from MX?; footprint (none) -> MX_Only:MXOnly-1U-Hotswap-Antishear
- MX12, MX42, MX54: renamed from MX?; footprint (none) -> MX_Only:MXOnly-1.25U-Hotswap
- MX24, MX36: renamed from MX?; footprint (none) -> MX_Only:MXOnly-2.75U-Hotswap
- MX3, MX80: renamed from MX?; footprint (none) -> MX_Only:MXOnly-1.5U-Hotswap
- MX4: renamed from MX?; footprint (none) -> MX_Only:MXOnly-1.75U-Hotswap
- MX5, MX79: renamed from MX?; footprint (none) -> MX_Only:MXOnly-2U-Hotswap
- MX71, MX76: renamed from MX?; footprint (none) -> MX_Only:MXOnly-2.25U-Hotswap
- R1, R2, R3, R4: footprint (none) -> R_0805_2012Metric
- R10, R11, R12, R13, R14, R15, R16, R17, R18, R19, R20, R21, R22, R5, R6, R7, R8, R9: renamed from R?; footprint (none) -> R_0805_2012Metric
- Y1: renamed from Y?; footprint (none) -> Crystal_SMD_3225-4pin_3.2x2.5mm
- gave numbers to parts that had none: 3
- renumbered U2 to U6
Connections:
- net 3.3V: now also C16.1, D4.1 (K), U3.3 (VI); no longer C1.1, C12.2, C2.1, C3.1, C4.1, C5.1, C6.1, C7.1, C8.1, J2.1 (VTref), U1.1 (VBAT), U1.24 (VDD), U1.36 (VDDIO2), U1.48 (VDD), U1.9 (VDDA)
- net 5V: now also R17.1; no longer C100.1, C101.1, C102.1, C103.1, C104.1, C105.1, C106.1, C107.1, C108.1, C109.1, C110.1, C111.1, C112.1, C113.1, C114.1, C115.1, C116.1, C117.1, C118.1, C119.1, C120.1, C121.1, C122.1, C123.1, C124.1, C125.1, C126.1, C127.1, C128.1, C129.1, C130.1, C131.1, C132.1, C133.1, C134.1, C135.1, C136.1, C137.1, C138.1, C139.1, C140.1, C141.1, C142.1, C145.1, C16.1, C47.1, C48.1, C49.1, C50.1, C51.1, C52.1, C53.1, C54.1, C55.1, C56.1, C57.1, C58.1, C59.1, C60.1, C61.1, C62.1, C63.1, C64.1, C65.1, C66.1, C67.1, C68.1, C69.1, C70.1, C71.1, C72.1, C73.1, C74.1, C75.1, C76.1, C77.1, C78.1, C79.1, C80.1, C81.1, C82.1, C83.1, C84.1, C85.1, C86.1, C87.1, C88.1, C89.1, C90.1, C91.1, C92.1, C93.1, C94.1, C95.1, C96.1, C97.1, C98.1, C99.1, D4.1 (K), LED1.1 (VCC), LED10.1 (VCC), LED11.1 (VCC), LED12.1 (VCC), LED13.1 (VCC), LED14.1 (VCC), LED15.1 (VCC), LED16.1 (VCC), LED17.1 (VCC), LED18.1 (VCC), LED19.1 (VCC), LED2.1 (VCC), LED20.1 (VCC), LED21.1 (VCC), LED22.1 (VCC), LED23.1 (VCC), LED24.1 (VCC), LED25.1 (VCC), LED26.1 (VCC), LED27.1 (VCC), LED28.1 (VCC), LED29.1 (VCC), LED3.1 (VCC), LED30.1 (VCC), LED31.1 (VCC), LED32.1 (VCC), LED33.1 (VCC), LED34.1 (VCC), LED35.1 (VCC), LED36.1 (VCC), LED37.1 (VCC), LED38.1 (VCC), LED39.1 (VCC), LED4.1 (VCC), LED40.1 (VCC), LED41.1 (VCC), LED42.1 (VCC), LED43.1 (VCC), LED44.1 (VCC), LED45.1 (VCC), LED46.1 (VCC), LED47.1 (VCC), LED48.1 (VCC), LED49.1 (VCC), LED5.1 (VCC), LED50.1 (VCC), LED51.1 (VCC), LED52.1 (VCC), LED53.1 (VCC), LED54.1 (VCC), LED55.1 (VCC), LED56.1 (VCC), LED57.1 (VCC), LED58.1 (VCC), LED59.1 (VCC), LED6.1 (VCC), LED60.1 (VCC), LED61.1 (VCC), LED62.1 (VCC), LED63.1 (VCC), LED64.1 (VCC), LED65.1 (VCC), LED66.1 (VCC), LED67.1 (VCC), LED68.1 (VCC), LED69.1 (VCC), LED7.1 (VCC), LED70.1 (VCC), LED71.1 (VCC), LED72.1 (VCC), LED73.1 (VCC), LED74.1 (VCC), LED75.1 (VCC), LED76.1 (VCC), LED77.1 (VCC), LED78.1 (VCC), LED79.1 (VCC), LED8.1 (VCC), LED80.1 (VCC), LED81.1 (VCC), LED82.1 (VCC), LED9.1 (VCC), U3.3 (VI)
- net D+: no longer U1.33 (PA12)
- net D-: no longer U1.32 (PA11)
- net GND: now also C143.2, C144.2, D5.2 (A), U5.1 (GND)
- net Keeb_D+: now also U1.33 (PA12)
- net Keeb_D-: now also U1.32 (PA11)
- net OUT1VBUS: now also F2.2
- net col3: now also MX42.1 (COL)
- net col4: now also MX54.1 (COL); no longer MX42.1 (COL)
- net col5: now also MX66.1 (COL); no longer MX54.1 (COL)
- net col6: no longer MX66.1 (COL)
- net row11: now also D42.1 (K), D54.1 (K), D66.1 (K), D78.1 (K); no longer D48.1 (K), D60.1 (K), D72.1 (K)
- net row12: now also D48.1 (K), D60.1 (K), D72.1 (K); no longer D42.1 (K), D54.1 (K), D66.1 (K), D78.1 (K)
- new net 5V_1000u: C100.1, C101.1, C102.1, C103.1, C104.1, C105.1, C106.1, C107.1, C108.1, C109.1, C110.1, C111.1, C112.1, C113.1, C114.1, C115.1, C116.1, C117.1, C118.1, C119.1, C120.1, C121.1, C122.1, C123.1, C124.1, C125.1, C126.1, C127.1, C128.1, C129.1, C130.1, C131.1, C132.1, C133.1, C134.1, C135.1, C136.1, C137.1, C138.1, C139.1, C140.1, C141.1, C142.1, C143.1, C145.1, C47.1, C48.1, C49.1, C50.1, C51.1, C52.1, C53.1, C54.1, C55.1, C56.1, C57.1, C58.1, C59.1, C60.1, C61.1, C62.1, C63.1, C64.1, C65.1, C66.1, C67.1, C68.1, C69.1, C70.1, C71.1, C72.1, C73.1, C74.1, C75.1, C76.1, C77.1, C78.1, C79.1, C80.1, C81.1, C82.1, C83.1, C84.1, C85.1, C86.1, C87.1, C88.1, C89.1, C90.1, C91.1, C92.1, C93.1, C94.1, C95.1, C96.1, C97.1, C98.1, C99.1, D5.1 (K), D6.1 (K), F2.1, LED1.1 (VCC), LED10.1 (VCC), LED11.1 (VCC), LED12.1 (VCC), LED13.1 (VCC), LED14.1 (VCC), LED15.1 (VCC), LED16.1 (VCC), LED17.1 (VCC), LED18.1 (VCC), LED19.1 (VCC), LED2.1 (VCC), LED20.1 (VCC), LED21.1 (VCC), LED22.1 (VCC), LED23.1 (VCC), LED24.1 (VCC), LED25.1 (VCC), LED26.1 (VCC), LED27.1 (VCC), LED28.1 (VCC), LED29.1 (VCC), LED3.1 (VCC), LED30.1 (VCC), LED31.1 (VCC), LED32.1 (VCC), LED33.1 (VCC), LED34.1 (VCC), LED35.1 (VCC), LED36.1 (VCC), LED37.1 (VCC), LED38.1 (VCC), LED39.1 (VCC), LED4.1 (VCC), LED40.1 (VCC), LED41.1 (VCC), LED42.1 (VCC), LED43.1 (VCC), LED44.1 (VCC), LED45.1 (VCC), LED46.1 (VCC), LED47.1 (VCC), LED48.1 (VCC), LED49.1 (VCC), LED5.1 (VCC), LED50.1 (VCC), LED51.1 (VCC), LED52.1 (VCC), LED53.1 (VCC), LED54.1 (VCC), LED55.1 (VCC), LED56.1 (VCC), LED57.1 (VCC), LED58.1 (VCC), LED59.1 (VCC), LED6.1 (VCC), LED60.1 (VCC), LED61.1 (VCC), LED62.1 (VCC), LED63.1 (VCC), LED64.1 (VCC), LED65.1 (VCC), LED66.1 (VCC), LED67.1 (VCC), LED68.1 (VCC), LED69.1 (VCC), LED7.1 (VCC), LED70.1 (VCC), LED71.1 (VCC), LED72.1 (VCC), LED73.1 (VCC), LED74.1 (VCC), LED75.1 (VCC), LED76.1 (VCC), LED77.1 (VCC), LED78.1 (VCC), LED79.1 (VCC), LED8.1 (VCC), LED80.1 (VCC), LED81.1 (VCC), LED82.1 (VCC), LED9.1 (VCC), U5.3 (VI)
- new net Keeb_3.3V: C1.1, C12.2, C144.1, C2.1, C3.1, C4.1, C5.1, C6.1, C7.1, C8.1, D6.2 (A), J2.1 (VTref), U1.1 (VBAT), U1.24 (VDD), U1.36 (VDDIO2), U1.48 (VDD), U1.9 (VDDA), U5.2 (VO)
Other:
- note added: "1.2V \nPower Supply"
- note added: "ARM CORTEX IC"
- note added: "Case ESD"
- note added: "Keeb ARM Chip Decoupling Caps"
- note added: "Keeb Power Supply"
- note added: "Key Matrix"
- note added: "Keyboard"
- note added: "Mounting Holes"
- note added: "RGB Matrix\nDecoupling Capacitors"
- note added: "Rotary Encoder"
- note added: "Serial Programmer"
- note added: "USB C IN"
- note added: "USB C OUT 1 (Top)"
- note added: "USB C Out 2 (Right)"
- note added: "USB C Out 3 (Left)"
- note added: "USB ESD Protection"
- note added: "USB HUB"
- note added: "USB Hub IC"
- note added: "USB Hub IC\nDecoupling Caps"
- note added: "USB Hub Power Output"
- note added: "USB Hub Voltage Supply\n"
- note added: "WS2812B RGB \nBacklight Matrix"
- moved on the sheet: C1, C10, C100, C101, C102, C103, C104, C105, C106, C107, C108, C109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
