File: Installation-01.sch (KiCad schematic (older format))
At the start: 461 parts, among them J2 Conn_ARM_JTAG_SWD_10, U1 STM32F072CBTx, U2 MCP1700-3302E_SOT23, U3 MCP1700-1202E_SOT23, U4 TUSB4041I, U5 MCP1700-3302E_SOT23, U6 USBLC6-2SC6, Y1 24MHz

Commit message: pcb diode start
Parts:
- gave numbers to parts that had none: 2
Changed lines of the file:
@@
 Connection ~ 16550 10650
 $Comp
-L power:GND #PWR?
+L power:GND #PWR04
 U 1 1 61A92AFB
 P 34650 6050
-F 0 "#PWR?" H 34650 5800 50  0001 C CNN
+F 0 "#PWR04" H 34650 5800 50  0001 C CNN
 F 1 "GND" V 34655 5922 50  0000 R CNN
 F 2 "" H 34650 6050 50  0001 C CNN
@@
 5V_RGB
 $Comp
-L ws2812b:WS2812B LED?
+L ws2812b:WS2812B LED86
 U 1 1 61A92B04
 P 34150 5850
-F 0 "LED?" H 34150 6337 60  0000 C CNN
+F 0 "LED86" H 34150 6337 60  0000 C CNN
 F 1 "right" H 34150 6231 60  0000 C CNN
 F 2 "WS2812B:WS2812B" V 34100 5850 60  0000 C CNN
@@
 	16050 5350 34800 5350
 $Comp
-L Device:C_Small C?
+L Device:C_Small C149
 U 1 1 61E0F33A
 P 16750 10800
-F 0 "C?" H 16842 10846 50  0000 L CNN
+F 0 "C149" H 16842 10846 50  0000 L CNN
 F 1 "0.1u" H 16842 10755 50  0000 L CNN
 F 2 "Capacitor_Tantalum_SMD:CP_EIA-2012-15_AVX-P" H 16750 10800 50  0001 C CNN

Commit message: pcb update
+key matrix and pcb components placed
+board outline
Parts:
- removed C134, C135, C136, C137, C138, C139, C140, C141, C142, C146, C147, C148, C149: 0.1u, Capacitor_Tantalum_SMD:CP_EIA-2012-15_AVX-P, symbol Device:C_Small
- MX1, MX10, MX11, MX13, MX14, MX15, MX16, MX17, MX18, MX19, MX2, MX20, MX21, MX22, MX23, MX25, MX26, MX27, MX28, MX29, MX31, MX32, MX33, MX34, MX35, MX37, MX38, MX39, MX40, MX41, MX43, MX44, MX45, MX46, MX47, MX48, MX49, MX50, MX51, MX52, MX53, MX55, MX56, MX57, MX58, MX59, MX60, MX61, MX62, MX63, MX64, MX65, MX66, MX67, MX68, MX69, MX7, MX70, MX72, MX73, MX74, MX75, MX77, MX78, MX8, MX81, MX82, MX83, MX84, MX9: footprint MX_Only:MXOnly-1U-Hotswap-Antishear -> MX_Only:MXOnly-1U-Hotswap
Connections:
- net at LED78.4 (DIN), LED85.2 (DOUT): no longer LED1.2 (DOUT)
- net at LED85.4 (DIN): now also LED1.2 (DOUT)
- no-connect marks 20 -> 26

Commit message: more pcb
Parts:
- MX6: footprint MX_Only:MXOnly-1.25U-Hotswap-Antishear -> MX_Only:MXOnly-1U-Hotswap
Changed lines of the file:
@@
 F 0 "MX6" H 25533 11023 60  0000 C CNN
 F 1 "Right Ctrl" H 25533 10949 20  0000 C CNN
-F 2 "MX_Only:MXOnly-1.25U-Hotswap-Antishear" H 24875 10775 60  0001 C CNN
+F 2 "MX_Only:MXOnly-1U-Hotswap" H 24875 10775 60  0001 C CNN
 F 3 "" H 24875 10775 60  0001 C CNN
 	1    25500 10800

Commit message: Added Acheron Lib
Parts:
- added LED87: LED, LED_THT:LED_D5.0mm, symbol Device:LED
- added R23: 68, Resistor_SMD:R_0805_2012Metric, symbol Device:R
- H1: footprint (none) -> MountingHole:MountingHole_2.7mm_M2.5_Pad
- H10, H2, H3, H4, H5, H6, H7, H8, H9: footprint (none) -> MountingHole:MountingHole_2.7mm_M2.5
- J2: footprint (none) -> Connector_PinSocket_1.00mm:PinSocket_2x05_P1.00mm_Vertical_SMD
Connections:
- net GND: now also R23.1
- net IndicatorLED: now reaches U1.38 (PA15)
- net IndicatorLED: now also LED87.2 (A)
- new net: LED87.1 (K), R23.2
- no-connect marks 26 -> 25
Other:
- note added: "Indicator LED"
Changed lines of the file:
@@
 F 0 "H1" V 20154 8000 50  0000 L CNN
 F 1 "MountingHole_Pad" V 20245 8000 50  0000 L CNN
-F 2 "" H 20200 7850 50  0001 C CNN
+F 2 "MountingHole:MountingHole_2.7mm_M2.5_Pad" H 20200 7850 50  0001 C CNN
 F 3 "~" H 20200 7850 50  0001 C CNN
 	1    20200 7850
@@
 F 0 "H2" H 20350 8096 50  0000 L CNN
 F 1 "MountingHole" H 20350 8005 50  0000 L CNN
-F 2 "" H 20250 8050 50  0001 C CNN
+F 2 "MountingHole:MountingHole_2.7mm_M2.5" H 20250 8050 50  0001 C CNN
 F 3 "~" H 20250 8050 50  0001 C CNN
 	1    20250 8050
@@
 F 0 "H3" H 20350 8296 50  0000 L CNN
 F 1 "MountingHole" H 20350 8205 50  0000 L CNN
-F 2 "" H 20250 8250 50  0001 C CNN
+F 2 "MountingHole:MountingHole_2.7mm_M2.5" H 20250 8250 50  0001 C CNN
 F 3 "~" H 20250 8250 50  0001 C CNN
 	1    20250 8250
@@
 F 0 "H4" H 20350 8496 50  0000 L CNN
 F 1 "MountingHole" H 20350 8405 50  0000 L CNN
-F 2 "" H 20250 8450 50  0001 C CNN
+F 2 "MountingHole:MountingHole_2.7mm_M2.5" H 20250 8450 50  0001 C CNN
 F 3 "~" H 20250 8450 50  0001 C CNN
 	1    20250 8450
@@
 F 0 "H5" H 20350 8696 50  0000 L CNN
 F 1 "MountingHole" H 20350 8605 50  0000 L CNN
-F 2 "" H 20250 8650 50  0001 C CNN
+F 2 "MountingHole:MountingHole_2.7mm_M2.5" H 20250 8650 50  0001 C CNN
 F 3 "~" H 20250 8650 50  0001 C CNN
 	1    20250 8650
@@
 F 0 "H6" H 20350 8896 50  0000 L CNN
 F 1 "MountingHole" H 20350 8805 50  0000 L CNN
-F 2 "" H 20250 8850 50  0001 C CNN
+F 2 "MountingHole:MountingHole_2.7mm_M2.5" H 20250 8850 50  0001 C CNN
 F 3 "~" H 20250 8850 50  0001 C CNN
 	1    20250 8850
@@
 F 0 "H7" H 20350 9096 50  0000 L CNN
 F 1 "MountingHole" H 20350 9005 50  0000 L CNN
-F 2 "" H 20250 9050 50  0001 C CNN
+F 2 "MountingHole:MountingHole_2.7mm_M2.5" H 20250 9050 50  0001 C CNN
 F 3 "~" H 20250 9050 50  0001 C CNN
 	1    20250 9050
@@
 F 0 "H8" H 20350 9296 50  0000 L CNN
 F 1 "MountingHole" H 20350 9205 50  0000 L CNN
-F 2 "" H 20250 9250 50  0001 C CNN
+F 2 "MountingHole:MountingHole_2.7mm_M2.5" H 20250 9250 50  0001 C CNN
 F 3 "~" H 20250 9250 50  0001 C CNN
 	1    20250 9250
@@
 F 0 "H9" H 20350 9496 50  0000 L CNN
 F 1 "MountingHole" H 20350 9405 50  0000 L CNN
-F 2 "" H 20250 9450 50  0001 C CNN
+F 2 "MountingHole:MountingHole_2.7mm_M2.5" H 20250 9450 50  0001 C CNN
 F 3 "~" H 20250 9450 50  0001 C CNN
 	1    20250 9450
@@
 F 0 "H10" H 20350 9696 50  0000 L CNN
 F 1 "MountingHole" H 20350 9605 50  0000 L CNN
-F 2 "" H 20250 9650 50  0001 C CNN
+F 2 "MountingHole:MountingHole_2.7mm_M2.5" H 20250 9650 50  0001 C CNN
 F 3 "~" H 20250 9650 50  0001 C CNN
 	1    20250 9650
@@
 F 0 "J2" H 23057 7596 50  0000 R CNN
 F 1 "Conn_ARM_JTAG_SWD_10" H 23057 7505 50  0000 R CNN
-F 2 "" H 23500 7550 50  0001 C CNN
+F 2 "Connector_PinSocket_1.00mm:PinSocket_2x05_P1.00mm_Vertical_SMD" H 23500 7550 50  0001 C CNN
 F 3 "http://infocenter.arm.com/help/topic/com.arm.doc.ddi0314h/DDI0314H_coresight_components_trm.pdf" V 23150 6300 50  0001 C CNN
 	1    23500 7550
@@
 NoConn ~ 17650 9150
 NoConn ~ 17650 9250
-NoConn ~ 19150 10950
 Wire Wire Line
 	16050 1750 35950 1750
+Text GLabel 19150 10950 2    50   Output ~ 0
+IndicatorLED
+Text GLabel 22150 10550 0    50   Input ~ 0
+IndicatorLED
+$Comp
+L Device:LED LED87
+U 1 1 5EBB66E8
+P 22300 10550
+F 0 "LED87" H 22293 10295 50  0000 C CNN
+F 1 "LED" H 22293 10386 50  0000 C CNN
+F 2 "LED_THT:LED_D5.0mm" H 22300 10550 50  0001 C CNN
+F 3 "~" H 22300 10550 50  0001 C CNN
+	1    22300 10550
+	-1   0    0    1
+$EndComp
+$Comp
+L Device:R R23
+U 1 1 5EBB6EE0
+P 22600 10550
+F 0 "R23" V 22393 10550 50  0000 C CNN
+F 1 "68" V 22484 10550 50  0000 C CNN
+F 2 "Resistor_SMD:R_0805_2012Metric" V 22530 10550 50  0001 C CNN
+F 3 "~" H 22600 10550 50  0001 C CNN
+	1    22600 10550
+	0    1    1    0
+$EndComp
+$Comp
+L power:GND #PWR05
+U 1 1 5EBBD97A
+P 22750 10550
+F 0 "#PWR05" H 22750 10300 50  0001 C CNN
+F 1 "GND" V 22755 10422 50  0000 R CNN
+F 2 "" H 22750 10550 50  0001 C CNN
+F 3 "" H 22750 10550 50  0001 C CNN
+	1    22750 10550
+	0    -1   -1   0
+$EndComp
+Wire Notes Line
+	21550 10200 21550 10700
+Wire Notes Line
+	21550 10700 23100 10700
+Wire Notes Line
+	23100 10700 23100 10200
+Wire Notes Line
+	23100 10200 21550 10200
+Text Notes 21600 10300 0    50   ~ 0
+Indicator LED
 $EndSCHEMATC

Commit message: pcb changes
Parts:
- H1: footprint MountingHole:MountingHole_2.7mm_M2.5_Pad -> acheron_MountingHoles:MoutingHole_Oval_7mm_5.0x2.5mm
- H10, H2, H5, H6, H7, H8, H9: footprint MountingHole:MountingHole_2.7mm_M2.5 -> acheron_MountingHoles:MoutingHole_Oval_7mm_5.0x2.5mm
- H3, H4: footprint MountingHole:MountingHole_2.7mm_M2.5 -> acheron_MountingHoles:halfSideHole
Changed lines of the file:
@@
 F 0 "H1" V 20154 8000 50  0000 L CNN
 F 1 "MountingHole_Pad" V 20245 8000 50  0000 L CNN
-F 2 "MountingHole:MountingHole_2.7mm_M2.5_Pad" H 20200 7850 50  0001 C CNN
+F 2 "acheron_MountingHoles:MoutingHole_Oval_7mm_5.0x2.5mm" H 20200 7850 50  0001 C CNN
 F 3 "~" H 20200 7850 50  0001 C CNN
 	1    20200 7850
@@
 F 0 "H2" H 20350 8096 50  0000 L CNN
 F 1 "MountingHole" H 20350 8005 50  0000 L CNN
-F 2 "MountingHole:MountingHole_2.7mm_M2.5" H 20250 8050 50  0001 C CNN
+F 2 "acheron_MountingHoles:MoutingHole_Oval_7mm_5.0x2.5mm" H 20250 8050 50  0001 C CNN
 F 3 "~" H 20250 8050 50  0001 C CNN
 	1    20250 8050
@@
 F 0 "H3" H 20350 8296 50  0000 L CNN
 F 1 "MountingHole" H 20350 8205 50  0000 L CNN
-F 2 "MountingHole:MountingHole_2.7mm_M2.5" H 20250 8250 50  0001 C CNN
+F 2 "acheron_MountingHoles:halfSideHole" H 20250 8250 50  0001 C CNN
 F 3 "~" H 20250 8250 50  0001 C CNN
 	1    20250 8250
@@
 F 0 "H4" H 20350 8496 50  0000 L CNN
 F 1 "MountingHole" H 20350 8405 50  0000 L CNN
-F 2 "MountingHole:MountingHole_2.7mm_M2.5" H 20250 8450 50  0001 C CNN
+F 2 "acheron_MountingHoles:halfSideHole" H 20250 8450 50  0001 C CNN
 F 3 "~" H 20250 8450 50  0001 C CNN
 	1    20250 8450
@@
 F 0 "H5" H 20350 8696 50  0000 L CNN
 F 1 "MountingHole" H 20350 8605 50  0000 L CNN
-F 2 "MountingHole:MountingHole_2.7mm_M2.5" H 20250 8650 50  0001 C CNN
+F 2 "acheron_MountingHoles:MoutingHole_Oval_7mm_5.0x2.5mm" H 20250 8650 50  0001 C CNN
 F 3 "~" H 20250 8650 50  0001 C CNN
 	1    20250 8650
@@
 F 0 "H6" H 20350 8896 50  0000 L CNN
 F 1 "MountingHole" H 20350 8805 50  0000 L CNN
-F 2 "MountingHole:MountingHole_2.7mm_M2.5" H 20250 8850 50  0001 C CNN
+F 2 "acheron_MountingHoles:MoutingHole_Oval_7mm_5.0x2.5mm" H 20250 8850 50  0001 C CNN
 F 3 "~" H 20250 8850 50  0001 C CNN
 	1    20250 8850
@@
 F 0 "H7" H 20350 9096 50  0000 L CNN
 F 1 "MountingHole" H 20350 9005 50  0000 L CNN
-F 2 "MountingHole:MountingHole_2.7mm_M2.5" H 20250 9050 50  0001 C CNN
+F 2 "acheron_MountingHoles:MoutingHole_Oval_7mm_5.0x2.5mm" H 20250 9050 50  0001 C CNN
 F 3 "~" H 20250 9050 50  0001 C CNN
 	1    20250 9050
@@
 F 0 "H8" H 20350 9296 50  0000 L CNN
 F 1 "MountingHole" H 20350 9205 50  0000 L CNN
-F 2 "MountingHole:MountingHole_2.7mm_M2.5" H 20250 9250 50  0001 C CNN
+F 2 "acheron_MountingHoles:MoutingHole_Oval_7mm_5.0x2.5mm" H 20250 9250 50  0001 C CNN
 F 3 "~" H 20250 9250 50  0001 C CNN
 	1    20250 9250
@@
 F 0 "H9" H 20350 9496 50  0000 L CNN
 F 1 "MountingHole" H 20350 9405 50  0000 L CNN
-F 2 "MountingHole:MountingHole_2.7mm_M2.5" H 20250 9450 50  0001 C CNN
+F 2 "acheron_MountingHoles:MoutingHole_Oval_7mm_5.0x2.5mm" H 20250 9450 50  0001 C CNN
 F 3 "~" H 20250 9450 50  0001 C CNN
 	1    20250 9450
@@
 F 0 "H10" H 20350 9696 50  0000 L CNN
 F 1 "MountingHole" H 20350 9605 50  0000 L CNN
-F 2 "MountingHole:MountingHole_2.7mm_M2.5" H 20250 9650 50  0001 C CNN
+F 2 "acheron_MountingHoles:MoutingHole_Oval_7mm_5.0x2.5mm" H 20250 9650 50  0001 C CNN
 F 3 "~" H 20250 9650 50  0001 C CNN
 	1    20250 9650
