File: Installation-01.kicad_pcb (KiCad board)
At the start: 2 copper layers, 433 parts, among them U1 STM32F072CBTx, U2 MCP1700-3302E_SOT23, U3 MCP1700-1202E_SOT23, U4 TUSB4041I, U5 MCP1700-3302E_SOT23, U6 USBLC6-2SC6

Commit message: pcb start
Parts:
- added Y1: 24MHz, Crystal:Crystal_SMD_3225-4Pin_3.2x2.5mm, F.Cu at (142.2, 203.8)
- MX1, MX10, MX11, MX13, MX14, MX15, MX16, MX17, MX18, MX19, MX2, MX20, MX21, MX22, MX23, MX25, MX26, MX27, MX28, MX29, MX31, MX32, MX33, MX34, MX35, MX37, MX38, MX39, MX40, MX41, MX43, MX44, MX45, MX46, MX47, MX48, MX49, MX50, MX51, MX52, MX53, MX55, MX56, MX57, MX58, MX59, MX6, MX60, MX61, MX62, MX63, MX64, MX65, MX66, MX67, MX68, MX69, MX7, MX70, MX72, MX73, MX74, MX75, MX77, MX78, MX8, MX81, MX82, MX9: footprint keyswitches:Kailh_socket_MX -> MX_Only:MXOnly-1U-Hotswap-Antishear
- moved MX80 320.3 mm to (277.8, 282.6)
- moved MX79 313.5 mm to (273.1, 263.5)
- moved MX21 273.0 mm to (82.5, 282.6)
- moved MX38 266.5 mm to (130.2, 263.5)
- moved MX34 260.2 mm to (-32.4, 166.4)
- moved MX15 258.2 mm to (63.5, 282.6)
- moved MX75 256.6 mm to (254.0, 282.6)
- moved MX7 252.1 mm to (41.3, 238.1)
- moved MX8 252.1 mm to (34.9, 263.5)
- moved MX69 240.3 mm to (234.9, 282.6)
- moved MX39 239.7 mm to (139.7, 282.6)
- moved MX9 238.9 mm to (44.5, 282.6)
- moved MX56 231.7 mm to (187.3, 263.5)
- moved MX26 230.1 mm to (92.1, 263.5)
- moved MX68 229.3 mm to (225.4, 263.5)
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