File: Installation-01.kicad_pcb (KiCad board)
At the start: 2 copper layers, 434 parts, among them U1 STM32F072CBTx, U2 MCP1700-3302E_SOT23, U3 MCP1700-1202E_SOT23, U4 TUSB4041I, U5 MCP1700-3302E_SOT23, U6 USBLC6-2SC6, Y1 24MHz

Commit message: continued pcb
Parts:
- moved MX76 345.0 mm to (270.7, 301.6)
- moved MX5 338.1 mm to (258.7, 320.7)
- moved MX4 297.9 mm to (23.0, 301.6)
- moved MX70 292.9 mm to (239.7, 301.6)
- moved MX59 288.7 mm to (211.1, 320.7)
- moved MX35 286.9 mm to (134.9, 320.7)
- moved MX46 278.2 mm to (163.5, 301.6)
- moved MX71 261.2 mm to (27.8, 320.7)
- moved MX53 259.2 mm to (192.1, 320.7)
- moved MX65 251.7 mm to (230.2, 320.7)
- moved MX11 243.0 mm to (58.7, 320.7)
- moved MX16 230.8 mm to (68.3, 301.6)
- moved MX29 229.0 mm to (115.9, 320.7)
- moved MX22 228.0 mm to (87.3, 301.6)
- moved MX64 227.6 mm to (220.7, 301.6)
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
Commit message: pcb
Parts:
- moved MX80 56.2 mm to (334.0, 281.9)
- moved MX10 1.64 mm to (49.2, 300.0)
- moved MX11 1.64 mm to (58.7, 319.0)
- moved MX15 1.64 mm to (63.5, 280.9)
- moved MX16 1.64 mm to (68.3, 300.0)
- moved MX17 1.64 mm to (77.8, 319.0)
- moved MX21 1.64 mm to (82.5, 280.9)
- moved MX22 1.64 mm to (87.3, 300.0)
- moved MX23 1.64 mm to (96.8, 319.0)
- moved MX27 1.64 mm to (101.6, 280.9)
- moved MX28 1.64 mm to (106.4, 300.0)
- moved MX29 1.64 mm to (115.9, 319.0)
- moved MX3 1.64 mm to (20.6, 280.9)
- moved MX33 1.64 mm to (120.7, 280.9)
- moved MX34 1.64 mm to (125.4, 300.0)
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Changed lines of the file:
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@@
   )
   (module MX_Only:MXOnly-1U-Hotswap-Antishear (layer F.Cu)
-    (at 254 282.575)
+    (at 254 280.9375)
     (fp_text reference MX75 (at 0 3.175) (layer Dwgs.User)
       (effects (font (size 1 1) (thickness 0.15)))
@@
   )
   (module MX_Only:MXOnly-1U-Hotswap-Antishear (layer F.Cu)
-    (at 239.7125 301.625)
+    (at 239.7125 299.9875)
     (fp_text reference MX70 (at 0 3.175) (layer Dwgs.User)
       (effects (font (size 1 1) (thickness 0.15)))
@@
   )
   (module MX_Only:MXOnly-1U-Hotswap-Antishear (layer F.Cu)
-    (at 234.95 282.575)
+    (at 234.95 280.9375)
     (fp_text reference MX69 (at 0 3.175) (layer Dwgs.User)
       (effects (font (size 1 1) (thickness 0.15)))
@@
   )
   (module MX_Only:MXOnly-1U-Hotswap-Antishear (layer F.Cu)
-    (at 230.1875 320.675)
+    (at 230.1875 319.0375)
     (fp_text reference MX65 (at 0 3.175) (layer Dwgs.User)
       (effects (font (size 1 1) (thickness 0.15)))
@@
   )
   (module MX_Only:MXOnly-1U-Hotswap-Antishear (layer F.Cu)
-    (at 220.6625 301.625)
+    (at 220.6625 299.9875)
     (fp_text reference MX64 (at 0 3.175) (layer Dwgs.User)
       (effects (font (size 1 1) (thickness 0.15)))
@@
   )
   (module MX_Only:MXOnly-1U-Hotswap-Antishear (layer F.Cu)
-    (at 215.9 282.575)
+    (at 215.9 280.9375)
     (fp_text reference MX63 (at 0 3.175) (layer Dwgs.User)
       (effects (font (size 1 1) (thickness 0.15)))
@@
   )
   (module MX_Only:MXOnly-1U-Hotswap-Antishear (layer F.Cu)
-    (at 211.1375 320.675)
+    (at 211.1375 319.0375)
     (fp_text reference MX59 (at 0 3.175) (layer Dwgs.User)
       (effects (font (size 1 1) (thickness 0.15)))
@@
   )
   (module MX_Only:MXOnly-1U-Hotswap-Antishear (layer F.Cu)
-    (at 201.6125 301.625)
+    (at 201.6125 299.9875)
     (fp_text reference MX58 (at 0 3.175) (layer Dwgs.User)
       (effects (font (size 1 1) (thickness 0.15)))
@@
   )
   (module MX_Only:MXOnly-1U-Hotswap-Antishear (layer F.Cu)
-    (at 196.85 282.575)
+    (at 196.85 280.9375)
     (fp_text reference MX57 (at 0 3.175) (layer Dwgs.User)
       (effects (font (size 1 1) (thickness 0.15)))
@@
   )
   (module MX_Only:MXOnly-1U-Hotswap-Antishear (layer F.Cu)
-    (at 192.0875 320.675)
+    (at 192.0875 319.0375)
     (fp_text reference MX53 (at 0 3.175) (layer Dwgs.User)
       (effects (font (size 1 1) (thickness 0.15)))
@@
   )
   (module MX_Only:MXOnly-1U-Hotswap-Antishear (layer F.Cu)
-    (at 182.5625 301.625)
+    (at 182.5625 299.9875)
     (fp_text reference MX52 (at 0 3.175) (layer Dwgs.User)
       (effects (font (size 1 1) (thickness 0.15)))
@@
   )
   (module MX_Only:MXOnly-1U-Hotswap-Antishear (layer F.Cu)
-    (at 177.8 282.575)
+    (at 177.8 280.9375)
     (fp_text reference MX51 (at 0 3.175) (layer Dwgs.User)
       (effects (font (size 1 1) (thickness 0.15)))
@@
   )
   (module MX_Only:MXOnly-1U-Hotswap-Antishear (layer F.Cu)
-    (at 173.0375 320.675)
+    (at 173.0375 319.0375)
     (fp_text reference MX47 (at 0 3.175) (layer Dwgs.User)
       (effects (font (size 1 1) (thickness 0.15)))
@@
   )
   (module MX_Only:MXOnly-1U-Hotswap-Antishear (layer F.Cu)
-    (at 163.5125 301.625)
+    (at 163.5125 299.9875)
     (fp_text reference MX46 (at 0 3.175) (layer Dwgs.User)
       (effects (font (size 1 1) (thickness 0.15)))
@@
   )
   (module MX_Only:MXOnly-1U-Hotswap-Antishear (layer F.Cu)
-    (at 158.75 282.575)
+    (at 158.75 280.9375)
     (fp_text reference MX45 (at 0 3.175) (layer Dwgs.User)
       (effects (font (size 1 1) (thickness 0.15)))
@@
   )
   (module MX_Only:MXOnly-1U-Hotswap-Antishear (layer F.Cu)
-    (at 153.9875 320.675)
+    (at 153.9875 319.0375)
     (fp_text reference MX41 (at 0 3.175) (layer Dwgs.User)
       (effects (font (size 1 1) (thickness 0.15)))
@@
   )
   (module MX_Only:MXOnly-1U-Hotswap-Antishear (layer F.Cu)
-    (at 144.4625 301.625)
+    (at 144.4625 299.9875)
     (fp_text reference MX40 (at 0 3.175) (layer Dwgs.User)
       (effects (font (size 1 1) (thickness 0.15)))
@@
   )
   (module MX_Only:MXOnly-1U-Hotswap-Antishear (layer F.Cu)
-    (at 139.7 282.575)
+    (at 139.7 280.9375)
     (fp_text reference MX39 (at 0 3.175) (layer Dwgs.User)
       (effects (font (size 1 1) (thickness 0.15)))
@@
   )
   (module MX_Only:MXOnly-1U-Hotswap-Antishear (layer F.Cu)
-    (at 134.9375 320.675)
+    (at 134.9375 319.0375)
     (fp_text reference MX35 (at 0 3.175) (layer Dwgs.User)
       (effects (font (size 1 1) (thickness 0.15)))
@@
   )
   (module MX_Only:MXOnly-1U-Hotswap-Antishear (layer F.Cu)
-    (at 125.4125 301.625)
+    (at 125.4125 299.9875)
     (fp_text reference MX34 (at 0 3.175) (layer Dwgs.User)
       (effects (font (size 1 1) (thickness 0.15)))
@@
   )
   (module MX_Only:MXOnly-1U-Hotswap-Antishear (layer F.Cu)
-    (at 120.65 282.575)
+    (at 120.65 280.9375)
     (fp_text reference MX33 (at 0 3.175) (layer Dwgs.User)
       (effects (font (size 1 1) (thickness 0.15)))
@@
   )
   (module MX_Only:MXOnly-1U-Hotswap-Antishear (layer F.Cu)
-    (at 115.8875 320.675)
+    (at 115.8875 319.0375)
     (fp_text reference MX29 (at 0 3.175) (layer Dwgs.User)
       (effects (font (size 1 1) (thickness 0.15)))
@@
   )
   (module MX_Only:MXOnly-1U-Hotswap-Antishear (layer F.Cu)
-    (at 106.3625 301.625)
+    (at 106.3625 299.9875)
     (fp_text reference MX28 (at 0 3.175) (layer Dwgs.User)
       (effects (font (size 1 1) (thickness 0.15)))
@@
   )
   (module MX_Only:MXOnly-1U-Hotswap-Antishear (layer F.Cu)
-    (at 101.6 282.575)
+    (at 101.6 280.9375)
     (fp_text reference MX27 (at 0 3.175) (layer Dwgs.User)
       (effects (font (size 1 1) (thickness 0.15)))
@@
   )
   (module MX_Only:MXOnly-1U-Hotswap-Antishear (layer F.Cu)
-    (at 96.8375 320.675)
+    (at 96.8375 319.0375)
     (fp_text reference MX23 (at 0 3.175) (layer Dwgs.User)
       (effects (font (size 1 1) (thickness 0.15)))
@@
   )
   (module MX_Only:MXOnly-1U-Hotswap-Antishear (layer F.Cu)
-    (at 87.3125 301.625)
+    (at 87.3125 299.9875)
     (fp_text reference MX22 (at 0 3.175) (layer Dwgs.User)
       (effects (font (size 1 1) (thickness 0.15)))
@@
   )
   (module MX_Only:MXOnly-1U-Hotswap-Antishear (layer F.Cu)
-    (at 82.55 282.575)
+    (at 82.55 280.9375)
     (fp_text reference MX21 (at 0 3.175) (layer Dwgs.User)
       (effects (font (size 1 1) (thickness 0.15)))
@@
   )
   (module MX_Only:MXOnly-1U-Hotswap-Antishear (layer F.Cu)
-    (at 77.7875 320.675)
+    (at 77.7875 319.0375)
     (fp_text reference MX17 (at 0 3.175) (layer Dwgs.User)
       (effects (font (size 1 1) (thickness 0.15)))
@@
   )
   (module MX_Only:MXOnly-1U-Hotswap-Antishear (layer F.Cu)
-    (at 68.2625 301.625)
+    (at 68.2625 299.9875)
     (fp_text reference MX16 (at 0 3.175) (layer Dwgs.User)
       (effects (font (size 1 1) (thickness 0.15)))
@@
   )
   (module MX_Only:MXOnly-1U-Hotswap-Antishear (layer F.Cu)
-    (at 63.5 282.575)
+    (at 63.5 280.9375)
     (fp_text reference MX15 (at 0 3.175) (layer Dwgs.User)
       (effects (font (size 1 1) (thickness 0.15)))
@@
   )
   (module MX_Only:MXOnly-1U-Hotswap-Antishear (layer F.Cu)
-    (at 58.7375 320.675)
+    (at 58.7375 319.0375)
     (fp_text reference MX11 (at 0 3.175) (layer Dwgs.User)
       (effects (font (size 1 1) (thickness 0.15)))
@@
   )
   (module MX_Only:MXOnly-1U-Hotswap-Antishear (layer F.Cu)
-    (at 49.2125 301.625)
+    (at 49.2125 299.9875)
     (fp_text reference MX10 (at 0 3.175) (layer Dwgs.User)
       (effects (font (size 1 1) (thickness 0.15)))
@@
   )
   (module MX_Only:MXOnly-1U-Hotswap-Antishear (layer F.Cu)
-    (at 44.45 282.575)
+    (at 44.45 280.9375)
     (fp_text reference MX9 (at 0 3.175) (layer Dwgs.User)
       (effects (font (size 1 1) (thickness 0.15)))
@@
   )
   (module MX_Only:MXOnly-1.5U-Hotswap (layer F.Cu)
-    (at 277.8125 282.575)
+    (at 334.01 281.94)
     (attr smd)
     (fp_text reference MX80 (at 0 3.048) (layer B.CrtYd)
@@
   )
   (module MX_Only:MXOnly-2.25U-Hotswap (layer F.Cu)
-    (at 270.66875 301.625)
+    (at 270.66875 299.9875)
     (attr smd)
     (fp_text reference MX76 (at 0 3.048) (layer B.CrtYd)
@@
   )
   (module MX_Only:MXOnly-2.25U-Hotswap (layer F.Cu)
-    (at 27.78125 320.675)
+    (at 27.78125 319.0375)
     (attr smd)
     (fp_text reference MX71 (at 0 3.048) (layer B.CrtYd)
@@
   )
   (module MX_Only:MXOnly-2U-Hotswap (layer F.Cu)
-    (at 258.7025 320.675)
+    (at 258.7025 319.0375)
     (attr smd)
     (fp_text reference MX5 (at 0 3.048) (layer B.CrtYd)
@@
   )
   (module MX_Only:MXOnly-1.75U-Hotswap (layer F.Cu)
-    (at 23.01875 301.625)
+    (at 23.01875 299.9875)
     (attr smd)
     (fp_text reference MX4 (at 0 3.048) (layer B.CrtYd)
@@
   )
   (module MX_Only:MXOnly-1.5U-Hotswap (layer F.Cu)
-    (at 20.6375 282.575)
+    (at 20.6375 280.9375)
     (attr smd)
     (fp_text reference MX3 (at 0 3.048) (layer B.CrtYd)

Commit message: pcb rgb finished
Parts:
- added C146: 0.1u, Capacitor_Tantalum_SMD:CP_EIA-2012-15_AVX-P, F.Cu at (63.5, 66.0)
- added C147: 0.1u, Capacitor_Tantalum_SMD:CP_EIA-2012-15_AVX-P, F.Cu at (68.0, 66.0)
- added C148: 0.1u, Capacitor_Tantalum_SMD:CP_EIA-2012-15_AVX-P, F.Cu at (72.5, 66.0)
- added C149: 0.1u, Capacitor_Tantalum_SMD:CP_EIA-2012-15_AVX-P, F.Cu at (62.5, 122.4)
- added D36: D, Diode_SMD:D_SOD-123, F.Cu at (177.8, 198.1)
- added D89: D, Diode_SMD:D_SOD-123, F.Cu at (64.1, 63.0)
- added D90: D, Diode_SMD:D_SOD-123, F.Cu at (69.9, 63.0)
- added LED83: down, WS2812B:WS2812B, F.Cu at (292.1, 348.7)
- added LED84: DEL, WS2812B:WS2812B, F.Cu at (282.7, 244.1)
- added LED85: Home, WS2812B:WS2812B, F.Cu at (316.2, 267.7)
- added LED86: right, WS2812B:WS2812B, F.Cu at (311.1, 348.7)
- added MX30: Space, MX_Only:MXOnly-6.25U-Hotswap, F.Cu at (137.1, 338.1)
- added MX83: Home, MX_Only:MXOnly-1U-Hotswap-Antishear, F.Cu at (315.9, 261.9)
- added MX84: End, MX_Only:MXOnly-1U-Hotswap-Antishear, F.Cu at (315.9, 280.9)
- LED1: value WS2812B -> ESC
- LED10: value WS2812B -> a
- LED11: value WS2812B -> z
- LED12: value WS2812B -> super
- LED13: value WS2812B -> F2
- LED14: value WS2812B -> 2
- LED15: value WS2812B -> w
- LED16: value WS2812B -> s
- LED17: value WS2812B -> x
- LED18: value WS2812B -> left alt
- LED19: value WS2812B -> F3
- LED2: value WS2812B -> `
- LED20: value WS2812B -> 3
- LED21: value WS2812B -> e
- LED22: value WS2812B -> d
- LED23: value WS2812B -> c
- LED24: value WS2812B -> space 1
- LED25: value WS2812B -> F4
- LED26: value WS2812B -> 4
- LED27: value WS2812B -> r
- LED28: value WS2812B -> f
- LED29: value WS2812B -> v
- LED3: value WS2812B -> tab
- LED30: value WS2812B -> space 2
- LED31: value WS2812B -> F5
- LED32: value WS2812B -> 5
- LED33: value WS2812B -> t
- LED34: value WS2812B -> g
- LED35: value WS2812B -> b
- LED36: value WS2812B -> space 3
- LED37: value WS2812B -> F6
- LED38: value WS2812B -> 6
- LED39: value WS2812B -> y
- LED4: value WS2812B -> caps
- LED40: value WS2812B -> h
- LED41: value WS2812B -> n
- LED42: value WS2812B -> space 4
- LED43: value WS2812B -> F7
- LED44: value WS2812B -> 7
- LED45: value WS2812B -> u
- LED46: value WS2812B -> j
- LED47: value WS2812B -> m
- LED48: value WS2812B -> space 5
- LED49: value WS2812B -> F8
- LED5: value WS2812B -> left shift
- LED50: value WS2812B -> 8
- LED51: value WS2812B -> i
- LED52: value WS2812B -> k
- LED53: value WS2812B -> ,
- LED54: value WS2812B -> right alt
- LED55: value WS2812B -> F9
- LED56: value WS2812B -> 9
- LED57: value WS2812B -> o
- LED58: value WS2812B -> l
- LED59: value WS2812B -> .
- LED6: value WS2812B -> left ctrl
- LED60: value WS2812B -> fn
- LED61: value WS2812B -> F10
- LED62: value WS2812B -> 0
- LED63: value WS2812B -> p
- LED64: value WS2812B -> ;
- LED65: value WS2812B -> /
- LED66: value WS2812B -> right ctrl
- LED67: value WS2812B -> F11
- LED68: value WS2812B -> -
- LED69: value WS2812B -> [
- LED7: value WS2812B -> F1
- LED70: value WS2812B -> '
- LED71: value WS2812B -> right shift
- LED72: value WS2812B -> left
- LED73: value WS2812B -> F12
- LED74: value WS2812B -> =
- LED75: value WS2812B -> ]
- LED76: value WS2812B -> enter
- LED77: value WS2812B -> up
- LED78: value WS2812B -> Backspace
- LED79: value WS2812B -> \
- LED8: value WS2812B -> 1
- LED80: value WS2812B -> page up
- LED81: value WS2812B -> page down
- LED82: value WS2812B -> End
- LED9: value WS2812B -> q
- MX6: footprint MX_Only:MXOnly-1U-Hotswap-Antishear -> MX_Only:MXOnly-1.25U-Hotswap
- moved LED12 384.1 mm to (41.9, 343.9), turned to 90 degrees
- moved LED4 357.9 mm to (23.1, 305.8), turned to 90 degrees
- moved MX24 351.5 mm to (170.7, 338.1)
- moved LED1 350.4 mm to (16.0, 244.1), turned to 90 degrees
- moved MX66 337.2 mm to (292.1, 342.9)
- moved LED29 335.3 mm to (115.8, 324.9), turned to 90 degrees
- moved LED11 332.2 mm to (58.7, 324.9), turned to 90 degrees
- moved MX72 330.6 mm to (311.1, 342.9)
- moved MX82 328.4 mm to (315.9, 319.0)
- moved MX77 327.4 mm to (292.1, 323.8)
- moved LED22 325.7 mm to (87.4, 305.8), turned to 90 degrees
- moved MX48 323.9 mm to (225.4, 338.1)
- moved MX6 322.3 mm to (246.9, 338.1)
- moved LED23 317.5 mm to (96.8, 324.9), turned to 90 degrees
- moved MX81 313.8 mm to (315.9, 300.0)
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Connections:
- net Net-(U1-Pad26) renamed E_Button2
- net Net-(U1-Pad27) renamed E_CCW2
- net Net-(U1-Pad28) renamed E_CW2
- C118 pad 2: Net-(C118-Pad2) -> GND
- D42 pad 1: row11 -> row12
- D48 pad 1: row12 -> row11
- D54 pad 1: row11 -> row12
- D60 pad 1: row12 -> row11
- D66 pad 1: row11 -> row12
- D72 pad 1: row12 -> row11
- D78 pad 1: row11 -> row12
- LED72 pad 4: Net-(LED5-Pad2) -> Net-(LED72-Pad4)
- MX42 pad 1: col3 -> col4
- MX54 pad 1: col4 -> col5
- MX66 pad 1: col5 -> col6
- R4 pad 2: Net-(LED73-Pad4) -> Net-(LED84-Pad4)
- U1 pad 17: E_CW -> col8
- U1 pad 29: E_CCW -> E_CW
- U1 pad 30: E_Button -> E_CCW
- U1 pad 31: Net-(U1-Pad31) -> E_Button

Commit message: pcb diode start
Parts:
- D13, D19, D25, D31, D37, D43, D7: moved to B.Cu
- moved D7 292.7 mm to (23.6, 238.3), turned to 90 degrees
- moved D19 288.8 mm to (71.4, 238.3), turned to 90 degrees
- moved D31 258.2 mm to (109.5, 238.3), turned to 90 degrees
- moved D25 235.3 mm to (90.4, 238.3), turned to 90 degrees
- moved D43 150.1 mm to (152.1, 238.3), turned to 90 degrees
- moved D13 109.7 mm to (52.3, 238.3), turned to 90 degrees
- moved D37 44.8 mm to (133.1, 238.3), turned to 90 degrees

Commit message: pcb update
+key matrix and pcb components placed
+board outline
Parts:
- removed C134, C135, C136, C137, C138, C139, C140, C141, C142, C146, C147, C148, C149: 0.1u, Capacitor_Tantalum_SMD:CP_EIA-2012-15_AVX-P
- C100, C101, C102, C103, C104, C105, C106, C107, C108, C109, C110, C111, C112, C113, C114, C115, C116, C117, C118, C119, C120, C121, C122, C123, C124, C125, C126, C127, C128, C129, C130, C131, C132, C133, C145, C47, C48, C49, C50, C51, C52, C53, C54, C55, C56, C57, C58, C59, C60, C61, C62, C63, C64, C65, C67, C68, C69, C70, C71, C72, C73, C74, C75, C76, C77, C78, C79, C80, C81, C82, C83, C84, C85, C86, C87, C88, C89, C90, C91, C92, C93, C94, C95, C96, C97, C98, C99, D10, D11, D12, D14, D15, D16, D17, D18, D20, D21, D22, D23, D24, D26, D27, D28, D29, D30, D32, D33, D34, D35, D36, D38, D39, D40, D41, D42, D44, D45, D46, D47, D48, D49, D50, D51, D52, D53, D54, D55, D56, D57, D58, D59, D60, D61, D62, D63, D64, D65, D66, D67, D68, D69, D70, D71, D72, D73, D74, D75, D76, D77, D78, D79, D8, D80, D81, D82, D83, D84, D85, D86, D87, D88, D89, D9, D90, R4: moved to B.Cu
- MX1, MX10, MX11, MX13, MX14, MX15, MX16, MX17, MX18, MX19, MX2, MX20, MX21, MX22, MX23, MX25, MX26, MX27, MX28, MX29, MX31, MX32, MX33, MX34, MX35, MX37, MX38, MX39, MX40, MX41, MX43, MX44, MX45, MX46, MX47, MX48, MX49, MX50, MX51, MX52, MX53, MX55, MX56, MX57, MX58, MX59, MX60, MX61, MX62, MX63, MX64, MX65, MX66, MX67, MX68, MX69, MX7, MX70, MX72, MX73, MX74, MX75, MX77, MX78, MX8, MX81, MX82, MX83, MX84, MX9: footprint MX_Only:MXOnly-1U-Hotswap-Antishear -> MX_Only:MXOnly-1U-Hotswap
- moved JIN1 415.7 mm to (-41.1, 219.2), turned to 180 degrees
- moved JOUT3 397.6 mm to (-50.8, 290.6), turned to 270 degrees
- moved D77 360.4 mm to (35.3, 319.0), turned to 90 degrees
- moved D90 334.5 mm to (323.6, 280.9), turned to 90 degrees
- moved D89 327.0 mm to (323.6, 261.9), turned to 90 degrees
- moved D78 312.7 mm to (318.8, 342.9), turned to 90 degrees
- moved D14 310.1 mm to (42.7, 261.9), turned to 90 degrees
- moved C124 309.6 mm to (225.3, 343.9), turned to 270 degrees
- moved D18 308.4 mm to (49.8, 338.1), turned to 90 degrees
- moved D17 306.0 mm to (66.3, 319.0), turned to 90 degrees
- moved D42 289.9 mm to (111.5, 338.1), turned to 90 degrees
- moved D66 285.6 mm to (280.7, 342.9), turned to 90 degrees
- moved D72 282.8 mm to (299.7, 342.9), turned to 90 degrees
- moved C132 273.0 mm to (41.9, 343.9), turned to 270 degrees
- moved D28 272.8 mm to (95.0, 300.0), turned to 90 degrees
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
Commit message: more pcb
Parts:
- MX6: footprint MX_Only:MXOnly-1.25U-Hotswap -> MX_Only:MXOnly-1U-Hotswap
- moved C126 5.59 mm to (190.5, 338.1)
- moved LED48 5.59 mm to (190.5, 338.1)
- moved C125 2.79 mm to (209.0, 343.9)
- moved C127 2.79 mm to (155.4, 338.1)
- moved LED42 2.79 mm to (155.4, 338.1)
- moved LED54 2.79 mm to (209.0, 343.9)
- moved C124 2.54 mm to (227.8, 343.9)
- moved D24 2.54 mm to (216.4, 338.1)
- moved D54 2.54 mm to (235.5, 338.1)
- moved LED60 2.54 mm to (227.8, 343.9)
- moved MX18 2.38 mm to (208.8, 338.1)
- moved MX24 2.38 mm to (173.0, 338.1)
- moved MX48 2.38 mm to (227.8, 338.1)
- moved D30 2.29 mm to (180.6, 338.1)
- moved C128 1.52 mm to (138.7, 343.7)
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Connections:
- LED78 pad 4: Net-(LED1-Pad2) -> Net-(LED78-Pad4)
- LED85 pad 2: Net-(LED1-Pad2) -> Net-(LED78-Pad4)
- LED85 pad 4: Net-(LED85-Pad4) -> Net-(LED1-Pad2)

Commit message: pcb changes
Parts:
- added H1: MountingHole_Pad, MountingHole:MountingHole_2.7mm_M2.5_Pad, F.Cu at (263.4, 145.8)
- added H10: MountingHole, MountingHole:MountingHole_2.7mm_M2.5, F.Cu at (291.2, 152.7)
- added H2: MountingHole, MountingHole:MountingHole_2.7mm_M2.5, F.Cu at (263.4, 152.7)
- added H3: MountingHole, MountingHole:MountingHole_2.7mm_M2.5, F.Cu at (270.3, 145.8)
- added H4: MountingHole, MountingHole:MountingHole_2.7mm_M2.5, F.Cu at (270.3, 152.7)
- added H5: MountingHole, MountingHole:MountingHole_2.7mm_M2.5, F.Cu at (277.3, 145.8)
- added H6: MountingHole, MountingHole:MountingHole_2.7mm_M2.5, F.Cu at (277.3, 152.7)
- added H7: MountingHole, MountingHole:MountingHole_2.7mm_M2.5, F.Cu at (284.2, 145.8)
- added H8: MountingHole, MountingHole:MountingHole_2.7mm_M2.5, F.Cu at (284.2, 152.7)
- added H9: MountingHole, MountingHole:MountingHole_2.7mm_M2.5, F.Cu at (291.2, 145.8)
- added J2: Conn_ARM_JTAG_SWD_10, Connector_PinSocket_1.00mm:PinSocket_2x05_P1.00mm_Vertical_SMD, F.Cu at (268.0, 163.8)
- added LED87: LED, LED_THT:LED_D5.0mm, F.Cu at (317.5, 237.7)
- added R23: 68, Resistor_SMD:R_0805_2012Metric, F.Cu at (316.2, 242.1)
Connections:
- U1 pad 38: Net-(U1-Pad38) -> IndicatorLED

Commit message: pcb
Parts:
- H1: footprint MountingHole:MountingHole_2.7mm_M2.5_Pad -> acheron_MountingHoles:MoutingHole_Oval_7mm_5.0x2.5mm
- H10, H2, H5, H6, H7, H8, H9: footprint MountingHole:MountingHole_2.7mm_M2.5 -> acheron_MountingHoles:MoutingHole_Oval_7mm_5.0x2.5mm
- H3, H4: footprint MountingHole:MountingHole_2.7mm_M2.5 -> acheron_MountingHoles:halfSideHole
- moved H4 30.3 mm to (299.7, 145.3)
- moved H10 28.0 mm to (306.2, 129.1)
- moved H2 28.0 mm to (278.4, 129.1)
- moved H6 28.0 mm to (292.3, 129.1)
- moved H8 28.0 mm to (299.2, 129.1)
- moved H9 27.3 mm to (306.9, 123.4)
- moved H1 27.3 mm to (279.1, 123.4)
- moved H5 27.3 mm to (293.0, 123.4)
- moved H7 27.3 mm to (300.0, 123.4)
