File: Peripherals/keyboard/Installation-01.kicad_pcb (KiCad board)
At the start: 2 copper layers, 448 parts, among them J2 Conn_ARM_JTAG_SWD_10, U1 STM32F072CBTx, U2 MCP1700-3302E_SOT23, U3 MCP1700-1202E_SOT23, U4 TUSB4041I, U5 MCP1700-3302E_SOT23, U6 USBLC6-2SC6, Y1 24MHz

Commit message: encoder
Parts:
- added E1: Rotary_Encoder_Switch_Chassis, acheron_Hardware:ALPS_EC11E, F.Cu at (-17.5, 261.9)
- added E2: Rotary_Encoder_Switch_Chassis, acheron_Hardware:ALPS_EC11E, F.Cu at (-17.5, 290.5)
Changed lines of the file:
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@@
     (tracks 0)
     (zones 0)
-    (modules 448)
+    (modules 450)
     (nets 301)
   )
@@
     (add_net row9)
   )
+  (module acheron_Hardware:ALPS_EC11E (layer F.Cu)
+    (at -17.4625 290.4625)
+    (fp_text reference E2 (at 0 0) (layer F.SilkS)
+      (effects (font (size 1 1) (thickness 0.15)))
+    )
+    (fp_text value Rotary_Encoder_Switch_Chassis (at 0 -2.5) (layer F.Fab)
+      (effects (font (size 1 1) (thickness 0.15)))
+    )
+    (fp_line (start 5.4 6.2) (end 3.2 6.2) (layer B.SilkS) (width 0.15))
+    (fp_line (start -5.4 6.2) (end -3.2 6.2) (layer B.SilkS) (width 0.15))
+    (fp_line (start -6.2 5.4) (end -6.2 2.4) (layer B.SilkS) (width 0.15))
+    (fp_line (start 6.2 5.4) (end 6.2 2.4) (layer B.SilkS) (width 0.15))
+    (fp_arc (start 5.4 5.4) (end 5.4 6.2) (angle -90) (layer B.SilkS) (width 0.15))
+    (fp_arc (start -5.4 5.4) (end -6.2 5.4) (angle -90) (layer B.SilkS) (width 0.15))
+    (fp_line (start 6.2 -2.4) (end 6.2 -5.4) (layer B.SilkS) (width 0.15))
+    (fp_arc (start 5.4 -5.4) (end 6.2 -5.4) (angle -90) (layer B.SilkS) (width 0.15))
+    (fp_line (start 5.4 -6.2) (end 3.2 -6.2) (layer B.SilkS) (width 0.15))
+    (fp_arc (start -5.4 -5.4) (end -5.4 -6.2) (angle -90) (layer B.SilkS) (width 0.15))
+    (fp_line (start -6.2 -2.4) (end -6.2 -5.4) (layer B.SilkS) (width 0.15))
+    (fp_line (start -5.4 -6.2) (end -3.4 -6.2) (layer B.SilkS) (width 0.15))
+    (fp_line (start 6 6) (end 4.2 6) (layer F.SilkS) (width 0.15))
+    (fp_line (start 3.2 -6) (end 6 -6) (layer F.SilkS) (width 0.15))
+    (fp_line (start 6 -6) (end 6 -2.4) (layer F.SilkS) (width 0.15))
+    (fp_line (start 6 6) (end 6 2.4) (layer F.SilkS) (width 0.15))
+    (fp_line (start -6 6) (end -6 2.4) (layer F.SilkS) (width 0.15))
+    (fp_line (start -6 -2.4) (end -6 -6) (layer F.SilkS) (width 0.15))
+    (fp_line (start 1 6) (end -6 6) (layer F.SilkS) (width 0.15))
+    (fp_line (start -6 -6) (end -3.4 -6) (layer F.SilkS) (width 0.15))
+    (pad "" connect oval (at 6.25 0) (size 1.651 2.7686) (layers B.Mask))
+    (pad "" connect oval (at -6.25 0) (size 1.651 2.7686) (layers B.Mask))
+    (pad "" smd circle (at 2.5 7.5) (size 1.016 1.016) (layers B.Mask))
+    (pad "" smd circle (at 0 7.5) (size 1.016 1.016) (layers B.Mask))
+    (pad "" smd circle (at -2.5 7.5) (size 1.016 1.016) (layers B.Mask))
+    (pad "" smd circle (at -2.5 -7) (size 1.016 1.016) (layers B.Mask))
+    (pad "" smd circle (at 2.5 -7) (size 1.016 1.016) (layers B.Mask))
+    (pad B thru_hole circle (at 2.5 7.5) (size 2.032 2.032) (drill 1.27) (layers *.Cu F.Mask)
+      (net 240 E_CW))
+    (pad A thru_hole circle (at -2.5 7.5) (size 2.032 2.032) (drill 1.27) (layers *.Cu F.Mask)
+      (net 234 E_CCW))
+    (pad C thru_hole circle (at 0 7.5) (size 2.032 2.032) (drill 1.27) (layers *.Cu F.Mask)
+      (net 1 GND))
+    (pad S1 thru_hole circle (at -2.5 -7) (size 2.032 2.032) (drill 1.27) (layers *.Cu F.Mask)
+      (net 233 E_Button))
+    (pad S2 thru_hole circle (at 2.5 -7) (size 2.032 2.032) (drill 1.27) (layers *.Cu F.Mask)
+      (net 1 GND))
+    (pad "" thru_hole oval (at -6.25 0) (size 2.799999 3.9) (drill oval 1.8 2.899999) (layers *.Cu F.Mask))
+    (pad "" thru_hole oval (at 6.25 0) (size 2.799999 3.9) (drill oval 1.8 2.899999) (layers *.Cu F.Mask))
+    (model ":Acheron 3D models:ALPS_EC11E.stp"
+      (offset (xyz 0.22 -0.06 10.25))
+      (scale (xyz 1 1 1))
+      (rotate (xyz 0 0 0))
+    )
+  )
+  (module acheron_Hardware:ALPS_EC11E (layer F.Cu)
+    (at -17.4625 261.8875)
+    (fp_text reference E1 (at 0 0) (layer F.SilkS)
+      (effects (font (size 1 1) (thickness 0.15)))
+    )
+    (fp_text value Rotary_Encoder_Switch_Chassis (at 0 -2.5) (layer F.Fab)
+      (effects (font (size 1 1) (thickness 0.15)))
+    )
+    (fp_line (start 5.4 6.2) (end 3.2 6.2) (layer B.SilkS) (width 0.15))
+    (fp_line (start -5.4 6.2) (end -3.2 6.2) (layer B.SilkS) (width 0.15))
+    (fp_line (start -6.2 5.4) (end -6.2 2.4) (layer B.SilkS) (width 0.15))
+    (fp_line (start 6.2 5.4) (end 6.2 2.4) (layer B.SilkS) (width 0.15))
+    (fp_arc (start 5.4 5.4) (end 5.4 6.2) (angle -90) (layer B.SilkS) (width 0.15))
+    (fp_arc (start -5.4 5.4) (end -6.2 5.4) (angle -90) (layer B.SilkS) (width 0.15))
+    (fp_line (start 6.2 -2.4) (end 6.2 -5.4) (layer B.SilkS) (width 0.15))
+    (fp_arc (start 5.4 -5.4) (end 6.2 -5.4) (angle -90) (layer B.SilkS) (width 0.15))
+    (fp_line (start 5.4 -6.2) (end 3.2 -6.2) (layer B.SilkS) (width 0.15))
+    (fp_arc (start -5.4 -5.4) (end -5.4 -6.2) (angle -90) (layer B.SilkS) (width 0.15))
+    (fp_line (start -6.2 -2.4) (end -6.2 -5.4) (layer B.SilkS) (width 0.15))
+    (fp_line (start -5.4 -6.2) (end -3.4 -6.2) (layer B.SilkS) (width 0.15))
+    (fp_line (start 6 6) (end 4.2 6) (layer F.SilkS) (width 0.15))
+    (fp_line (start 3.2 -6) (end 6 -6) (layer F.SilkS) (width 0.15))
+    (fp_line (start 6 -6) (end 6 -2.4) (layer F.SilkS) (width 0.15))
+    (fp_line (start 6 6) (end 6 2.4) (layer F.SilkS) (width 0.15))
+    (fp_line (start -6 6) (end -6 2.4) (layer F.SilkS) (width 0.15))
+    (fp_line (start -6 -2.4) (end -6 -6) (layer F.SilkS) (width 0.15))
+    (fp_line (start 1 6) (end -6 6) (layer F.SilkS) (width 0.15))
+    (fp_line (start -6 -6) (end -3.4 -6) (layer F.SilkS) (width 0.15))
+    (pad "" connect oval (at 6.25 0) (size 1.651 2.7686) (layers B.Mask))
+    (pad "" connect oval (at -6.25 0) (size 1.651 2.7686) (layers B.Mask))
+    (pad "" smd circle (at 2.5 7.5) (size 1.016 1.016) (layers B.Mask))
+    (pad "" smd circle (at 0 7.5) (size 1.016 1.016) (layers B.Mask))
+    (pad "" smd circle (at -2.5 7.5) (size 1.016 1.016) (layers B.Mask))
+    (pad "" smd circle (at -2.5 -7) (size 1.016 1.016) (layers B.Mask))
+    (pad "" smd circle (at 2.5 -7) (size 1.016 1.016) (layers B.Mask))
+    (pad B thru_hole circle (at 2.5 7.5) (size 2.032 2.032) (drill 1.27) (layers *.Cu F.Mask)
+      (net 284 E_CW2))
+    (pad A thru_hole circle (at -2.5 7.5) (size 2.032 2.032) (drill 1.27) (layers *.Cu F.Mask)
+      (net 285 E_CCW2))
+    (pad C thru_hole circle (at 0 7.5) (size 2.032 2.032) (drill 1.27) (layers *.Cu F.Mask)
+      (net 1 GND))
+    (pad S1 thru_hole circle (at -2.5 -7) (size 2.032 2.032) (drill 1.27) (layers *.Cu F.Mask)
+      (net 286 E_Button2))
+    (pad S2 thru_hole circle (at 2.5 -7) (size 2.032 2.032) (drill 1.27) (layers *.Cu F.Mask)
+      (net 1 GND))
+    (pad "" thru_hole oval (at -6.25 0) (size 2.799999 3.9) (drill oval 1.8 2.899999) (layers *.Cu F.Mask))
+    (pad "" thru_hole oval (at 6.25 0) (size 2.799999 3.9) (drill oval 1.8 2.899999) (layers *.Cu F.Mask))
+    (model ":Acheron 3D models:ALPS_EC11E.stp"
+      (offset (xyz 0.22 -0.06 10.25))
+      (scale (xyz 1 1 1))
+      (rotate (xyz 0 0 0))
+    )
+  )
   (module acheron_MountingHoles:MoutingHole_Oval_7mm_5.0x2.5mm (layer F.Cu)

Commit message: keyboard
Parts:
- added LED88: LED, LED_SMD:LED_0805_2012Metric, F.Cu at (320.7, 238.1)
- added R24: 68, Resistor_SMD:R_0805_2012Metric, F.Cu at (320.8, 241.7)
- LED87: footprint LED_THT:LED_D5.0mm -> LED_SMD:LED_0805_2012Metric
- U6: moved to B.Cu
- moved U1 320.3 mm to (-25.4, 238.8)
- moved C12 270.2 mm to (-31.2, 233.9), turned to 270 degrees
- moved C42 266.6 mm to (-43.9, 229.1), turned to 90 degrees
- moved U6 179.4 mm to (-41.1, 229.4), turned to 90 degrees
- moved LED87 6.36 mm to (311.1, 238.1)
- moved R23 5.09 mm to (311.1, 241.7)
Connections:
- U1 pad 2: Net-(U1-Pad2) -> capsLockLED
Other:
- board text added: "Caps"
- board text added: "Power"

Commit message: some bs with power management on pcb
Parts:
- C10, C9: moved to B.Cu
- moved F1 324.7 mm to (-35.4, 239.5), turned to 180 degrees
- moved R2 298.8 mm to (-29.5, 230.4), turned to 90 degrees
- moved R3 292.4 mm to (-25.4, 230.4), turned to 270 degrees
- moved C9 282.9 mm to (-29.6, 242.3)
- moved R1 268.7 mm to (-31.8, 230.4), turned to 90 degrees
- moved C10 262.0 mm to (-27.7, 239.7), turned to 270 degrees
- moved C11 243.4 mm to (-27.4, 230.4), turned to 270 degrees
- moved U2 148.5 mm to (-30.5, 239.5), turned to 180 degrees
- moved D1 99.1 mm to (-29.7, 245.4)
- moved D2 84.0 mm to (-33.0, 236.5)
- moved KEEBSWITCH1 72.7 mm to (-1.52, 189.5)
- moved JOUT3 22.7 mm to (-41.1, 270.0)
- moved C12 17.8 mm to (-14.5, 240.0)
- moved U1 17.8 mm to (-8.64, 244.9)
- moved JIN1 8.89 mm to (-32.3, 219.2)
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