File: Peripherals/keyboard-v1/Installation-01.kicad_pcb (KiCad board)
At the start: 2 copper layers, 386 parts, among them J2 Conn_ARM_JTAG_SWD_10, U1 STM32F072CBTx, U5 MCP1700-3302E_SOT23, U6 USBLC6-2SC6

Commit message: v1 board
Parts:
- removed C66: 0.1u, Capacitor_Tantalum_SMD:CP_EIA-2012-15_AVX-P
- moved H1 331.8 mm to (-30.5, 4.01)
- moved J2 312.6 mm to (-9.11, 19.1), turned to 180 degrees
- moved R18 310.5 mm to (-31.5, 9.66), turned to 270 degrees
- moved C143 310.3 mm to (-17.3, 6.99), turned to 180 degrees
- moved C20 305.1 mm to (-29.0, 9.66), turned to 270 degrees
- moved C3 303.4 mm to (-26.1, 31.4), turned to 270 degrees
- moved C7 299.8 mm to (-31.2, 23.8), turned to 180 degrees
- moved C8 296.8 mm to (-31.2, 26.3), turned to 180 degrees
- moved C6 295.8 mm to (-16.0, 26.3)
- moved F2 293.2 mm to (-12.2, 9.55)
- moved C1 290.7 mm to (-21.0, 31.4), turned to 270 degrees
- moved C2 288.4 mm to (-23.6, 31.4), turned to 270 degrees
- moved C4 285.0 mm to (-16.0, 21.2)
- moved C144 273.1 mm to (-22.4, 9.55), turned to 90 degrees
- moved C5 271.0 mm to (-16.0, 23.8)
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Other:
- board outline added: 376.5 x 138 mm

Commit message: border
Other:
- board size 376.5 x 138 mm -> 428.6 x 233.3 mm

Commit message: finished pcb
Parts:
- removed H1: MountingHole_Pad, acheron_MountingHoles:MoutingHole_Oval_7mm_5.0x2.5mm
- removed H10, H2, H5, H6, H7, H8, H9: MountingHole, acheron_MountingHoles:MoutingHole_Oval_7mm_5.0x2.5mm
- removed H3, H4: MountingHole, acheron_MountingHoles:halfSideHole
- U6: moved to F.Cu
- moved C11 23.7 mm to (-16.9, 18.6)
- moved R2 23.7 mm to (-19.0, 18.6)
- moved R3 23.7 mm to (-14.9, 18.6)
- moved R1 23.7 mm to (-21.3, 18.6)
- moved C1 22.9 mm to (1.56, 27.6)
- moved C12 22.9 mm to (-8.60, 17.4)
- moved C2 22.9 mm to (-0.98, 27.6)
- moved C4 22.9 mm to (6.64, 17.4)
- moved C5 22.9 mm to (6.64, 19.9)
- moved C6 22.9 mm to (6.64, 22.5)
- moved C7 22.9 mm to (-8.60, 19.9)
- moved C8 22.9 mm to (-8.60, 22.5)
- moved U1 22.9 mm to (-0.98, 19.9)
- moved C3 22.9 mm to (-3.52, 27.6)
- moved C20 21.2 mm to (-15.4, 25.9)
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Other:
- board size 428.6 x 233.3 mm -> 367 x 138 mm

Commit message: added 3d models
3d models for components and pcb
plate svg n stuff
Parts:
- D3, D6, J2, JIN1: moved to B.Cu
- LED1, LED10, LED11, LED12, LED13, LED14, LED15, LED16, LED17, LED18, LED19, LED2, LED20, LED21, LED22, LED23, LED24, LED25, LED26, LED27, LED28, LED29, LED3, LED30, LED31, LED32, LED33, LED34, LED35, LED36, LED37, LED38, LED39, LED4, LED40, LED41, LED42, LED43, LED44, LED45, LED46, LED47, LED48, LED49, LED5, LED50, LED51, LED52, LED53, LED54, LED55, LED56, LED57, LED58, LED59, LED6, LED60, LED61, LED62, LED63, LED64, LED65, LED66, LED67, LED68, LED69, LED7, LED70, LED71, LED72, LED73, LED74, LED75, LED76, LED77, LED78, LED79, LED8, LED80, LED81, LED82, LED83, LED84, LED85, LED86, LED9: footprint WS2812B:WS2812B -> WS2812B:LED_SK6812MINI_PLCC4_3.5x3.5mm_P1.75mm
- moved E1 3.00 mm to (-9.64, 42.7)
- moved E2 3.00 mm to (-9.64, 71.3)
- moved C42 2.00 mm to (-3.26, 11.6)
- moved U6 2.00 mm to (0.12, 11.6)
- moved J2 1.98 mm to (-8.50, 26.5), turned to 0 degrees
- moved D3 1.94 mm to (-22.0, 23.5)
- moved C20 1.58 mm to (-14.9, 24.4)
- moved R18 1.58 mm to (-17.4, 24.4)
- turned JIN1 to 0 degrees
Connections:
- LED1 pad 1: 5V_1000u -> Net-(LED1-Pad1)
- LED1 pad 2: Net-(LED1-Pad2) -> GND
- LED1 pad 3: GND -> Net-(LED1-Pad3)
- LED1 pad 4: Net-(LED1-Pad4) -> 5V_1000u
- LED10 pad 1: 5V_1000u -> Net-(LED10-Pad1)
- LED10 pad 2: Net-(LED10-Pad2) -> GND
- LED10 pad 3: GND -> Net-(LED10-Pad3)
- LED10 pad 4: Net-(LED10-Pad4) -> 5V_1000u
- LED11 pad 1: 5V_1000u -> Net-(LED11-Pad1)
- LED11 pad 2: Net-(LED11-Pad2) -> GND
- LED11 pad 3: GND -> Net-(LED11-Pad3)
- LED11 pad 4: Net-(LED11-Pad4) -> 5V_1000u
- LED12 pad 1: 5V_1000u -> Net-(LED12-Pad1)
- LED12 pad 2: Net-(LED12-Pad2) -> GND
- LED12 pad 3: GND -> Net-(LED12-Pad3)
- LED12 pad 4: Net-(LED12-Pad4) -> 5V_1000u
- LED13 pad 1: 5V_1000u -> Net-(LED13-Pad1)
- LED13 pad 2: Net-(LED13-Pad2) -> GND
- LED13 pad 3: GND -> Net-(LED13-Pad3)
- LED13 pad 4: Net-(LED13-Pad4) -> 5V_1000u
- LED14 pad 1: 5V_1000u -> Net-(LED14-Pad1)
- LED14 pad 2: Net-(LED14-Pad2) -> GND
- LED14 pad 3: GND -> Net-(LED14-Pad3)
- LED14 pad 4: Net-(LED14-Pad4) -> 5V_1000u
- LED15 pad 1: 5V_1000u -> Net-(LED15-Pad1)
- LED15 pad 2: Net-(LED15-Pad2) -> GND
- LED15 pad 3: GND -> Net-(LED15-Pad3)
- LED15 pad 4: Net-(LED15-Pad4) -> 5V_1000u
- LED16 pad 1: 5V_1000u -> Net-(LED10-Pad3)
- LED16 pad 2: Net-(LED10-Pad4) -> GND
- LED16 pad 3: GND -> Net-(LED16-Pad3)
- LED16 pad 4: Net-(LED16-Pad4) -> 5V_1000u
- LED17 pad 1: 5V_1000u -> Net-(LED11-Pad3)
- LED17 pad 2: Net-(LED11-Pad4) -> GND
- LED17 pad 3: GND -> Net-(LED17-Pad3)
- LED17 pad 4: Net-(LED17-Pad4) -> 5V_1000u
- LED18 pad 1: 5V_1000u -> Net-(LED12-Pad3)
- LED18 pad 2: Net-(LED12-Pad4) -> GND
- LED18 pad 3: GND -> Net-(LED18-Pad3)
- LED18 pad 4: Net-(LED18-Pad4) -> 5V_1000u
- LED19 pad 1: 5V_1000u -> Net-(LED13-Pad3)
- LED19 pad 2: Net-(LED13-Pad4) -> GND
- LED19 pad 3: GND -> Net-(LED19-Pad3)
- LED19 pad 4: Net-(LED19-Pad4) -> 5V_1000u
- LED2 pad 1: 5V_1000u -> Net-(LED2-Pad1)
- LED2 pad 2: Net-(LED2-Pad2) -> GND
- LED2 pad 3: GND -> Net-(LED2-Pad3)
- LED2 pad 4: Net-(LED2-Pad4) -> 5V_1000u
- LED20 pad 1: 5V_1000u -> Net-(LED14-Pad3)
- LED20 pad 2: Net-(LED14-Pad4) -> GND
- LED20 pad 3: GND -> Net-(LED20-Pad3)
- LED20 pad 4: Net-(LED20-Pad4) -> 5V_1000u
- LED21 pad 1: 5V_1000u -> Net-(LED15-Pad3)
- LED21 pad 2: Net-(LED15-Pad4) -> GND
- LED21 pad 3: GND -> Net-(LED21-Pad3)
- LED21 pad 4: Net-(LED21-Pad4) -> 5V_1000u
- LED22 pad 1: 5V_1000u -> Net-(LED16-Pad3)
- LED22 pad 2: Net-(LED16-Pad4) -> GND
- LED22 pad 3: GND -> Net-(LED22-Pad3)
- LED22 pad 4: Net-(LED22-Pad4) -> 5V_1000u
- LED23 pad 1: 5V_1000u -> Net-(LED17-Pad3)
- LED23 pad 2: Net-(LED17-Pad4) -> GND
- LED23 pad 3: GND -> Net-(LED23-Pad3)
- LED23 pad 4: Net-(LED23-Pad4) -> 5V_1000u
- LED24 pad 1: 5V_1000u -> Net-(LED18-Pad3)
- LED24 pad 2: Net-(LED18-Pad4) -> GND
- LED24 pad 3: GND -> Net-(LED24-Pad3)
- LED24 pad 4: Net-(LED24-Pad4) -> 5V_1000u
- LED25 pad 1: 5V_1000u -> Net-(LED19-Pad3)
- LED25 pad 2: Net-(LED19-Pad4) -> GND
- LED25 pad 3: GND -> Net-(LED25-Pad3)
- LED25 pad 4: Net-(LED25-Pad4) -> 5V_1000u
- LED26 pad 1: 5V_1000u -> Net-(LED20-Pad3)
- LED26 pad 2: Net-(LED20-Pad4) -> GND
- LED26 pad 3: GND -> Net-(LED26-Pad3)
- LED26 pad 4: Net-(LED26-Pad4) -> 5V_1000u
- LED27 pad 1: 5V_1000u -> Net-(LED21-Pad3)
- LED27 pad 2: Net-(LED21-Pad4) -> GND
- LED27 pad 3: GND -> Net-(LED27-Pad3)
- LED27 pad 4: Net-(LED27-Pad4) -> 5V_1000u
- LED28 pad 1: 5V_1000u -> Net-(LED22-Pad3)
- LED28 pad 2: Net-(LED22-Pad4) -> GND
- LED28 pad 3: GND -> Net-(LED28-Pad3)
- LED28 pad 4: Net-(LED28-Pad4) -> 5V_1000u
- LED29 pad 1: 5V_1000u -> Net-(LED23-Pad3)
- LED29 pad 2: Net-(LED23-Pad4) -> GND
- LED29 pad 3: GND -> Net-(LED29-Pad3)
- LED29 pad 4: Net-(LED29-Pad4) -> 5V_1000u
- LED3 pad 1: 5V_1000u -> Net-(LED3-Pad1)
- LED3 pad 2: Net-(LED3-Pad2) -> GND
- LED3 pad 3: GND -> Net-(LED3-Pad3)
- LED3 pad 4: Net-(LED3-Pad4) -> 5V_1000u
- LED30 pad 1: 5V_1000u -> Net-(LED24-Pad3)
- LED30 pad 2: Net-(LED24-Pad4) -> GND
- LED30 pad 3: GND -> Net-(LED30-Pad3)
- LED30 pad 4: Net-(LED30-Pad4) -> 5V_1000u
- LED31 pad 1: 5V_1000u -> Net-(LED25-Pad3)
- LED31 pad 2: Net-(LED25-Pad4) -> GND
- LED31 pad 3: GND -> Net-(LED31-Pad3)
- LED31 pad 4: Net-(LED31-Pad4) -> 5V_1000u
- LED32 pad 1: 5V_1000u -> Net-(LED26-Pad3)
- LED32 pad 2: Net-(LED26-Pad4) -> GND
- LED32 pad 3: GND -> Net-(LED32-Pad3)
- LED32 pad 4: Net-(LED32-Pad4) -> 5V_1000u
- LED33 pad 1: 5V_1000u -> Net-(LED27-Pad3)
- LED33 pad 2: Net-(LED27-Pad4) -> GND
- LED33 pad 3: GND -> Net-(LED33-Pad3)
- LED33 pad 4: Net-(LED33-Pad4) -> 5V_1000u
- LED34 pad 1: 5V_1000u -> Net-(LED28-Pad3)
- LED34 pad 2: Net-(LED28-Pad4) -> GND
- LED34 pad 3: GND -> Net-(LED34-Pad3)
- LED34 pad 4: Net-(LED34-Pad4) -> 5V_1000u
- LED35 pad 1: 5V_1000u -> Net-(LED29-Pad3)
- LED35 pad 2: Net-(LED29-Pad4) -> GND
- LED35 pad 3: GND -> Net-(LED35-Pad3)
- LED35 pad 4: Net-(LED35-Pad4) -> 5V_1000u
- LED36 pad 1: 5V_1000u -> Net-(LED30-Pad3)
- LED36 pad 2: Net-(LED30-Pad4) -> GND
- LED36 pad 3: GND -> Net-(LED36-Pad3)
- LED36 pad 4: Net-(LED36-Pad4) -> 5V_1000u
- LED37 pad 1: 5V_1000u -> Net-(LED31-Pad3)
- LED37 pad 2: Net-(LED31-Pad4) -> GND
- LED37 pad 3: GND -> Net-(LED37-Pad3)
- LED37 pad 4: Net-(LED37-Pad4) -> 5V_1000u
- LED38 pad 1: 5V_1000u -> Net-(LED32-Pad3)
- LED38 pad 2: Net-(LED32-Pad4) -> GND
- LED38 pad 3: GND -> Net-(LED38-Pad3)
- LED38 pad 4: Net-(LED38-Pad4) -> 5V_1000u
- LED39 pad 1: 5V_1000u -> Net-(LED33-Pad3)
- LED39 pad 2: Net-(LED33-Pad4) -> GND
- LED39 pad 3: GND -> Net-(LED39-Pad3)
- LED39 pad 4: Net-(LED39-Pad4) -> 5V_1000u
- LED4 pad 1: 5V_1000u -> Net-(LED4-Pad1)
- LED4 pad 2: Net-(LED4-Pad2) -> GND
- LED4 pad 3: GND -> Net-(LED10-Pad1)
- LED4 pad 4: Net-(LED10-Pad2) -> 5V_1000u
- LED40 pad 1: 5V_1000u -> Net-(LED34-Pad3)
- LED40 pad 2: Net-(LED34-Pad4) -> GND
- LED40 pad 3: GND -> Net-(LED40-Pad3)
- LED40 pad 4: Net-(LED40-Pad4) -> 5V_1000u
- LED41 pad 1: 5V_1000u -> Net-(LED35-Pad3)
- LED41 pad 2: Net-(LED35-Pad4) -> GND
- LED41 pad 3: GND -> Net-(LED41-Pad3)
- LED41 pad 4: Net-(LED41-Pad4) -> 5V_1000u
- LED42 pad 1: 5V_1000u -> Net-(LED36-Pad3)
- LED42 pad 2: Net-(LED36-Pad4) -> GND
- LED42 pad 3: GND -> Net-(LED42-Pad3)
- LED42 pad 4: Net-(LED42-Pad4) -> 5V_1000u
- LED43 pad 1: 5V_1000u -> Net-(LED37-Pad3)
- LED43 pad 2: Net-(LED37-Pad4) -> GND
- LED43 pad 3: GND -> Net-(LED43-Pad3)
- LED43 pad 4: Net-(LED43-Pad4) -> 5V_1000u
- LED44 pad 1: 5V_1000u -> Net-(LED38-Pad3)
- LED44 pad 2: Net-(LED38-Pad4) -> GND
- LED44 pad 3: GND -> Net-(LED44-Pad3)
- LED44 pad 4: Net-(LED44-Pad4) -> 5V_1000u
- LED45 pad 1: 5V_1000u -> Net-(LED39-Pad3)
- LED45 pad 2: Net-(LED39-Pad4) -> GND
- LED45 pad 3: GND -> Net-(LED45-Pad3)
- LED45 pad 4: Net-(LED45-Pad4) -> 5V_1000u
- LED46 pad 1: 5V_1000u -> Net-(LED40-Pad3)
- LED46 pad 2: Net-(LED40-Pad4) -> GND
- LED46 pad 3: GND -> Net-(LED46-Pad3)
- LED46 pad 4: Net-(LED46-Pad4) -> 5V_1000u
- LED47 pad 1: 5V_1000u -> Net-(LED41-Pad3)
- LED47 pad 2: Net-(LED41-Pad4) -> GND
- LED47 pad 3: GND -> Net-(LED47-Pad3)
- LED47 pad 4: Net-(LED47-Pad4) -> 5V_1000u
- LED48 pad 1: 5V_1000u -> Net-(LED42-Pad3)
- LED48 pad 2: Net-(LED42-Pad4) -> GND
- LED48 pad 3: GND -> Net-(LED48-Pad3)
- LED48 pad 4: Net-(LED48-Pad4) -> 5V_1000u
- LED49 pad 1: 5V_1000u -> Net-(LED43-Pad3)
- LED49 pad 2: Net-(LED43-Pad4) -> GND
- LED49 pad 3: GND -> Net-(LED49-Pad3)
- LED49 pad 4: Net-(LED49-Pad4) -> 5V_1000u
- LED5 pad 1: 5V_1000u -> Net-(LED5-Pad1)
- LED5 pad 2: Net-(LED5-Pad2) -> GND
- LED5 pad 3: GND -> Net-(LED11-Pad1)
- LED5 pad 4: Net-(LED11-Pad2) -> 5V_1000u
- LED50 pad 1: 5V_1000u -> Net-(LED44-Pad3)
- LED50 pad 2: Net-(LED44-Pad4) -> GND
- LED50 pad 3: GND -> Net-(LED50-Pad3)
- LED50 pad 4: Net-(LED50-Pad4) -> 5V_1000u
- LED51 pad 1: 5V_1000u -> Net-(LED45-Pad3)
- LED51 pad 2: Net-(LED45-Pad4) -> GND
- LED51 pad 3: GND -> Net-(LED51-Pad3)
- LED51 pad 4: Net-(LED51-Pad4) -> 5V_1000u
- LED52 pad 1: 5V_1000u -> Net-(LED46-Pad3)
- LED52 pad 2: Net-(LED46-Pad4) -> GND
- LED52 pad 3: GND -> Net-(LED52-Pad3)
- LED52 pad 4: Net-(LED52-Pad4) -> 5V_1000u
- LED53 pad 1: 5V_1000u -> Net-(LED47-Pad3)
- LED53 pad 2: Net-(LED47-Pad4) -> GND
- LED53 pad 3: GND -> Net-(LED53-Pad3)
- LED53 pad 4: Net-(LED53-Pad4) -> 5V_1000u
- LED54 pad 1: 5V_1000u -> Net-(LED48-Pad3)
- LED54 pad 2: Net-(LED48-Pad4) -> GND
- LED54 pad 3: GND -> Net-(LED54-Pad3)
- LED54 pad 4: Net-(LED54-Pad4) -> 5V_1000u
- LED55 pad 1: 5V_1000u -> Net-(LED49-Pad3)
- LED55 pad 2: Net-(LED49-Pad4) -> GND
- LED55 pad 3: GND -> Net-(LED55-Pad3)
- LED55 pad 4: Net-(LED55-Pad4) -> 5V_1000u
- LED56 pad 1: 5V_1000u -> Net-(LED50-Pad3)
- LED56 pad 2: Net-(LED50-Pad4) -> GND
- LED56 pad 3: GND -> Net-(LED56-Pad3)
- LED56 pad 4: Net-(LED56-Pad4) -> 5V_1000u
- LED57 pad 1: 5V_1000u -> Net-(LED51-Pad3)
- LED57 pad 2: Net-(LED51-Pad4) -> GND
- LED57 pad 3: GND -> Net-(LED57-Pad3)
- LED57 pad 4: Net-(LED57-Pad4) -> 5V_1000u
- LED58 pad 1: 5V_1000u -> Net-(LED52-Pad3)
- LED58 pad 2: Net-(LED52-Pad4) -> GND
- LED58 pad 3: GND -> Net-(LED58-Pad3)
- LED58 pad 4: Net-(LED58-Pad4) -> 5V_1000u
- LED59 pad 1: 5V_1000u -> Net-(LED53-Pad3)
- LED59 pad 2: Net-(LED53-Pad4) -> GND
- LED59 pad 3: GND -> Net-(LED59-Pad3)
- LED59 pad 4: Net-(LED59-Pad4) -> 5V_1000u
- LED6 pad 1: 5V_1000u -> Net-(LED6-Pad1)
- LED6 pad 2: Net-(LED6-Pad2) -> GND
- LED6 pad 3: GND -> Net-(LED12-Pad1)
- LED6 pad 4: Net-(LED12-Pad2) -> 5V_1000u
- LED60 pad 1: 5V_1000u -> Net-(LED54-Pad3)
- LED60 pad 2: Net-(LED54-Pad4) -> GND
- LED60 pad 3: GND -> Net-(LED60-Pad3)
- LED60 pad 4: Net-(LED60-Pad4) -> 5V_1000u
- LED61 pad 1: 5V_1000u -> Net-(LED55-Pad3)
- LED61 pad 2: Net-(LED55-Pad4) -> GND
- LED61 pad 3: GND -> Net-(LED61-Pad3)
- LED61 pad 4: Net-(LED61-Pad4) -> 5V_1000u
- LED62 pad 1: 5V_1000u -> Net-(LED56-Pad3)
- LED62 pad 2: Net-(LED56-Pad4) -> GND
- LED62 pad 3: GND -> Net-(LED62-Pad3)
- LED62 pad 4: Net-(LED62-Pad4) -> 5V_1000u
- LED63 pad 1: 5V_1000u -> Net-(LED57-Pad3)
- LED63 pad 2: Net-(LED57-Pad4) -> GND
- LED63 pad 3: GND -> Net-(LED63-Pad3)
- LED63 pad 4: Net-(LED63-Pad4) -> 5V_1000u
- LED64 pad 1: 5V_1000u -> Net-(LED58-Pad3)
- LED64 pad 2: Net-(LED58-Pad4) -> GND
- LED64 pad 3: GND -> Net-(LED64-Pad3)
- LED64 pad 4: Net-(LED64-Pad4) -> 5V_1000u
- LED65 pad 1: 5V_1000u -> Net-(LED59-Pad3)
- LED65 pad 2: Net-(LED59-Pad4) -> GND
- LED65 pad 3: GND -> Net-(LED65-Pad3)
- LED65 pad 4: Net-(LED65-Pad4) -> 5V_1000u
- LED66 pad 1: 5V_1000u -> Net-(LED60-Pad3)
- LED66 pad 2: Net-(LED60-Pad4) -> GND
- LED66 pad 3: GND -> Net-(LED66-Pad3)
- LED66 pad 4: Net-(LED66-Pad4) -> 5V_1000u
- LED67 pad 1: 5V_1000u -> Net-(LED61-Pad3)
- LED67 pad 2: Net-(LED61-Pad4) -> GND
- LED67 pad 3: GND -> Net-(LED67-Pad3)
- LED67 pad 4: Net-(LED67-Pad4) -> 5V_1000u
- LED68 pad 1: 5V_1000u -> Net-(LED62-Pad3)
- LED68 pad 2: Net-(LED62-Pad4) -> GND
- LED68 pad 3: GND -> Net-(LED68-Pad3)
- LED68 pad 4: Net-(LED68-Pad4) -> 5V_1000u
- LED69 pad 1: 5V_1000u -> Net-(LED63-Pad3)
- LED69 pad 2: Net-(LED63-Pad4) -> GND
- LED69 pad 3: GND -> Net-(LED69-Pad3)
- LED69 pad 4: Net-(LED69-Pad4) -> 5V_1000u
- LED7 pad 1: 5V_1000u -> Net-(LED1-Pad3)
- LED7 pad 2: Net-(LED1-Pad4) -> GND
- LED7 pad 3: GND -> Net-(LED13-Pad1)
- LED7 pad 4: Net-(LED13-Pad2) -> 5V_1000u
- LED70 pad 1: 5V_1000u -> Net-(LED64-Pad3)
- LED70 pad 2: Net-(LED64-Pad4) -> GND
- LED70 pad 3: GND -> Net-(LED70-Pad3)
- LED70 pad 4: Net-(LED70-Pad4) -> 5V_1000u
- LED71 pad 1: 5V_1000u -> Net-(LED65-Pad3)
- LED71 pad 2: Net-(LED65-Pad4) -> GND
- LED71 pad 3: GND -> Net-(LED71-Pad3)
- LED71 pad 4: Net-(LED71-Pad4) -> 5V_1000u
- LED72 pad 1: 5V_1000u -> Net-(LED66-Pad3)
- LED72 pad 2: Net-(LED66-Pad4) -> GND
- LED72 pad 3: GND -> Net-(LED72-Pad3)
- LED72 pad 4: Net-(LED72-Pad4) -> 5V_1000u
- LED73 pad 1: 5V_1000u -> Net-(LED67-Pad3)
- LED73 pad 2: Net-(LED67-Pad4) -> GND
- LED73 pad 3: GND -> Net-(LED73-Pad3)
- LED73 pad 4: Net-(LED73-Pad4) -> 5V_1000u
- LED74 pad 1: 5V_1000u -> Net-(LED68-Pad3)
- LED74 pad 2: Net-(LED68-Pad4) -> GND
- LED74 pad 3: GND -> Net-(LED74-Pad3)
- LED74 pad 4: Net-(LED74-Pad4) -> 5V_1000u
- LED75 pad 1: 5V_1000u -> Net-(LED69-Pad3)
- LED75 pad 2: Net-(LED69-Pad4) -> GND
- LED75 pad 3: GND -> Net-(LED75-Pad3)
- LED75 pad 4: Net-(LED75-Pad4) -> 5V_1000u
- LED76 pad 1: 5V_1000u -> Net-(LED70-Pad3)
- LED76 pad 2: Net-(LED70-Pad4) -> GND
- LED76 pad 3: GND -> Net-(LED76-Pad3)
- LED76 pad 4: Net-(LED76-Pad4) -> 5V_1000u
- LED77 pad 1: 5V_1000u -> Net-(LED71-Pad3)
- LED77 pad 2: Net-(LED71-Pad4) -> GND
- LED77 pad 3: GND -> Net-(LED77-Pad3)
- LED77 pad 4: Net-(LED77-Pad4) -> 5V_1000u
- LED78 pad 1: 5V_1000u -> Net-(LED74-Pad3)
- LED78 pad 2: Net-(LED74-Pad4) -> GND
- LED78 pad 3: GND -> Net-(LED78-Pad3)
- LED78 pad 4: Net-(LED78-Pad4) -> 5V_1000u
- LED79 pad 1: 5V_1000u -> Net-(LED75-Pad3)
- LED79 pad 2: Net-(LED75-Pad4) -> GND
- LED79 pad 3: GND -> Net-(LED79-Pad3)
- LED79 pad 4: Net-(LED79-Pad4) -> 5V_1000u
- LED8 pad 1: 5V_1000u -> Net-(LED2-Pad3)
- LED8 pad 2: Net-(LED2-Pad4) -> GND
- LED8 pad 3: GND -> Net-(LED14-Pad1)
- LED8 pad 4: Net-(LED14-Pad2) -> 5V_1000u
- LED80 pad 1: 5V_1000u -> Net-(LED76-Pad3)
- LED80 pad 2: Net-(LED76-Pad4) -> GND
- LED80 pad 3: GND -> Net-(LED3-Pad1)
- LED80 pad 4: Net-(LED3-Pad2) -> 5V_1000u
- LED81 pad 1: 5V_1000u -> Net-(LED77-Pad3)
- LED81 pad 2: Net-(LED77-Pad4) -> GND
- LED81 pad 3: GND -> Net-(LED4-Pad1)
- LED81 pad 4: Net-(LED4-Pad2) -> 5V_1000u
- LED82 pad 1: 5V_1000u -> Net-(LED79-Pad3)
- LED82 pad 2: Net-(LED79-Pad4) -> GND
- LED82 pad 3: GND -> Net-(LED2-Pad1)
- LED82 pad 4: Net-(LED2-Pad2) -> 5V_1000u
- LED83 pad 1: 5V_1000u -> Net-(LED72-Pad3)
- LED83 pad 2: Net-(LED72-Pad4) -> GND
- LED83 pad 3: GND -> Net-(LED83-Pad3)
- LED83 pad 4: Net-(LED83-Pad4) -> 5V_1000u
- LED84 pad 1: 5V_1000u -> Net-(LED73-Pad3)
- LED84 pad 2: Net-(LED73-Pad4) -> GND
- LED84 pad 3: GND -> Net-(LED84-Pad3)
- LED84 pad 4: Net-(LED84-Pad4) -> 5V_1000u
- LED85 pad 1: 5V_1000u -> Net-(LED78-Pad3)
- LED85 pad 2: Net-(LED78-Pad4) -> GND
- LED85 pad 3: GND -> Net-(LED1-Pad1)
- LED85 pad 4: Net-(LED1-Pad2) -> 5V_1000u
- LED86 pad 1: 5V_1000u -> Net-(LED83-Pad3)
- LED86 pad 2: Net-(LED83-Pad4) -> GND
- LED86 pad 3: GND -> Net-(LED5-Pad1)
- LED86 pad 4: Net-(LED5-Pad2) -> 5V_1000u
- LED9 pad 1: 5V_1000u -> Net-(LED3-Pad3)
- LED9 pad 2: Net-(LED3-Pad4) -> GND
- LED9 pad 3: GND -> Net-(LED15-Pad1)
- LED9 pad 4: Net-(LED15-Pad2) -> 5V_1000u
- R4 pad 2: Net-(LED84-Pad4) -> Net-(LED84-Pad3)
Other:
- board size 367 x 138 mm -> 370 x 138 mm
