File: Peripherals/keyboard-v1/Installation-01.kicad_pcb (KiCad board)
At the start: 2 copper layers, 370 x 138 mm, 375 parts, among them J2 Conn_ARM_JTAG_SWD_10, U1 STM32F072CBTx, U5 MCP1700-3302E_SOT23, U6 USBLC6-2SC6

Commit message: bruh moment
Parts:
- moved C1 23.5 mm to (-16.2, 12.2), turned to 180 degrees
- moved C6 23.0 mm to (-16.3, 21.2), turned to 180 degrees
- moved C5 22.9 mm to (-16.3, 19.4), turned to 180 degrees
- moved C4 22.9 mm to (-16.3, 17.6), turned to 180 degrees
- moved C2 20.4 mm to (-16.2, 14.0), turned to 180 degrees
- moved C42 17.8 mm to (-21.1, 11.4), turned to 180 degrees
- moved C3 17.3 mm to (-16.2, 15.8), turned to 180 degrees
- moved D3 17.1 mm to (-35.0, 12.4), turned to 180 degrees
- moved C20 12.9 mm to (-21.1, 13.2), turned to 0 degrees
- moved C12 12.7 mm to (-21.1, 15.0), turned to 180 degrees
- moved D6 9.07 mm to (-8.00, 5.20), turned to 270 degrees
- moved C7 8.26 mm to (-16.3, 23.0)
- moved C8 8.02 mm to (-16.3, 24.8)
- moved C144 7.58 mm to (-11.4, 9.00), turned to 180 degrees
- moved J2 7.53 mm to (-6.73, 19.2)
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Connections:
- MX5 pad 1: col1 -> col7
- MX54 pad 1: col5 -> col1
- MX6 pad 1: col1 -> col7
- MX71 pad 1: col6 -> col1
Routing:
- net GND: track 0.00 -> 57.8 mm, vias 0 -> 2
- net Keeb_3.3V: track 0.00 -> 32.3 mm, vias 0 -> 2
- net VBUS: track 0.00 -> 16.6 mm, vias 0 -> 3
- net 5V_1000u: track 0.00 -> 11.5 mm
- net Net-(D27-Pad2): track 0.00 -> 4.41 mm
- net Net-(D15-Pad2): track 0.00 -> 4.41 mm
- net Net-(D31-Pad2): track 0.00 -> 4.40 mm
- net Net-(D25-Pad2): track 0.00 -> 4.40 mm
- net Net-(D13-Pad2): track 0.00 -> 4.40 mm
- net Net-(D19-Pad2): track 0.00 -> 4.40 mm
- net Net-(D84-Pad2): track 0.00 -> 4.35 mm
- net Net-(D7-Pad2): track 0.00 -> 4.35 mm
- net Net-(D67-Pad2): track 0.00 -> 4.35 mm
- net Net-(D61-Pad2): track 0.00 -> 4.35 mm
- net Net-(D79-Pad2): track 0.00 -> 4.35 mm
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Other:
- rule trace_min: 0.2 -> 0.127
- rule via_min_size: 0.4 -> 0.6
