File: Peripherals/keyboard-v1/Installation-01.sch (KiCad schematic (older format))
At the start: 450 parts, among them J2 Conn_ARM_JTAG_SWD_10, U1 STM32F072CBTx, U2 MCP1700-3302E_SOT23, U3 MCP1700-1202E_SOT23, U4 TUSB4041I, U5 MCP1700-3302E_SOT23, U6 USBLC6-2SC6, Y1 24MHz

Commit message: version change
-added bleeding edge project
-added version 1 project
Parts:
- removed C10, C16, C19, C9: 100n, Capacitor_Tantalum_SMD:CP_EIA-2012-15_AVX-P, symbol Device:C_Small
- removed C13, C14, C15: 4.7n, Capacitor_Tantalum_SMD:CP_EIA-2012-15_AVX-P, symbol Device:C_Small
- removed C17, C18: 10p, Capacitor_Tantalum_SMD:CP_EIA-2012-15_AVX-P, symbol Device:C_Small
- removed C21, C22, C23, C24, C25, C26, C27, C28, C29, C31, C32, C34, C35, C36, C37, C38, C39, C40, C41: 0.1u, Capacitor_Tantalum_SMD:CP_EIA-2012-15_AVX-P, symbol Device:C_Small
- removed C30, C33: 10u, Capacitor_Tantalum_SMD:CP_EIA-2012-15_AVX-P, symbol Device:C_Small
- removed C43, C44, C45, C46: 150u, Capacitor_Tantalum_SMD:CP_EIA-2012-15_AVX-P, symbol Device:C_Small
- removed D1: B260, Diode_SMD:D_SMB, symbol Diode:B260
- removed D2, D4: 1N914, Diode_THT:D_DO-35_SOD27_P7.62mm_Horizontal, symbol Diode:1N914
- removed F1: Polyfuse_Small, Fuse:Fuse_1206_3216Metric, symbol Device:Polyfuse_Small
- removed JOUT1, JOUT2, JOUT3: USB_C_Receptacle_USB2.0, Type-C:USB_C_GCT_USB4085, symbol Connector:USB_C_Receptacle_USB2.0
- removed KEEBSWITCH1, OUTSWITCH1, OUTSWITCH2, OUTSWITCH3: TPS2001CDGNR, TPS2001CDGNR:TPS2001CDGNR, symbol TPS2001CDGNR:TPS2001CDGNR
- removed R10, R11, R12, R13, R8, R9: 5.1k, Resistor_SMD:R_0805_2012Metric, symbol Device:R_Small
- removed R14: 10M, Resistor_SMD:R_0805_2012Metric, symbol Device:R_Small
- removed R15, R19, R20, R21, R22: 10k, Resistor_SMD:R_0805_2012Metric, symbol Device:R_Small
- removed R16: 9.53k, Resistor_SMD:R_0805_2012Metric, symbol Device:R_Small
- removed R17: 90.9k, Resistor_SMD:R_0805_2012Metric, symbol Device:R_Small
- removed R5, R6, R7: 22k, Resistor_SMD:R_0805_2012Metric, symbol Device:R_Small
- removed U2: MCP1700-3302E_SOT23, Package_TO_SOT_SMD:SOT-23, symbol Regulator_Linear:MCP1700-3302E_SOT23
- removed U3: MCP1700-1202E_SOT23, Package_TO_SOT_SMD:SOT-23, symbol Regulator_Linear:MCP1700-1202E_SOT23
- removed U4: TUSB4041I, Package_QFP:HTQFP-64-1EP_10x10mm_P0.5mm_EP8x8mm_Mask4.4x4.4mm_ThermalVias, symbol Interface_USB:TUSB4041I
- removed Y1: 24MHz, Crystal:Crystal_SMD_3225-4Pin_3.2x2.5mm, symbol Device:Crystal
- added LED88: LED, LED_SMD:LED_0805_2012Metric, symbol Device:LED
- added R24: 68, Resistor_SMD:R_0805_2012Metric, symbol Device:R
- LED87: footprint LED_THT:LED_D5.0mm -> LED_SMD:LED_0805_2012Metric
- U6: symbol Power_Protection:USBLC6-2SC6 -> Installation-01-rescue:USBLC6-2SC6-Power_Protection
Connections:
- net labels added: capsLockLED
- net labels removed: 1.2V, 3.3V, 5V, DOUT1+, DOUT1-, DOUT2+, DOUT2-, DOUT3+, DOUT3-, Keeb_D+, Keeb_D-, OUT1VBUS, OUT2VBUS, OUT3VBUS, OVERCUR1, OVERCUR2, OVERCUR3, OVERCUR4, PWRCTL1, PWRCTL2, PWRCTL3, PWRCTL4, VDD33_USB, VDD_USB
- wire segments 1178 -> 866
- no-connect marks 25 -> 9
Other:
- note added: "Caps Lock LED"
- note removed: "1.2V \nPower Supply"
- note removed: "USB C OUT 1 (Top)"
- note removed: "USB C Out 2 (Right)"
- note removed: "USB C Out 3 (Left)"
- note removed: "USB HUB"
- note removed: "USB Hub IC"
- note removed: "USB Hub IC\nDecoupling Caps"
- note removed: "USB Hub Power Output"
- note removed: "USB Hub Voltage Supply\n"
- moved on the sheet: C11, C20, C42, D3, JIN1, R1, R18, R2, R3

Commit message: v1 board
Parts:
- removed C66: 0.1u, Capacitor_Tantalum_SMD:CP_EIA-2012-15_AVX-P, symbol Device:C_Small
Connections:
- wire segments 866 -> 864
Changed lines of the file:
@@
 $EndComp
 $Comp
-L Device:C_Small C66
-U 1 1 617DD98B
-P 15850 10050
-F 0 "C66" H 15942 10096 50  0000 L CNN
-F 1 "0.1u" H 15942 10005 50  0000 L CNN
-F 2 "Capacitor_Tantalum_SMD:CP_EIA-2012-15_AVX-P" H 15850 10050 50  0001 C CNN
-F 3 "~" H 15850 10050 50  0001 C CNN
-	1    15850 10050
-	0    1    1    0
-$EndComp
-$Comp
-L Device:C_Small C67
-U 1 1 617DD991
-P 15850 10200
-F 0 "C67" H 15942 10246 50  0000 L CNN
-F 1 "0.1u" H 15942 10155 50  0000 L CNN
-F 2 "Capacitor_Tantalum_SMD:CP_EIA-2012-15_AVX-P" H 15850 10200 50  0001 C CNN
-F 3 "~" H 15850 10200 50  0001 C CNN
-	1    15850 10200
-	0    1    1    0
-$EndComp
-$Comp
 L Device:C_Small C68
 U 1 1 617DD997
@@
 	15950 9900 15950 9750
 Wire Wire Line
-	15950 10050 15950 9900
-Wire Wire Line
-	15950 10200 15950 10050
-Wire Wire Line
-	15950 10350 15950 10200
-Wire Wire Line
 	15950 10500 15950 10350
 Wire Wire Line
@@
 	15750 9750 15750 9900
 Wire Wire Line
-	15750 9900 15750 10050
-Wire Wire Line
-	15750 10050 15750 10200
-Wire Wire Line
-	15750 10200 15750 10350
-Wire Wire Line
 	15750 10350 15750 10500
 Wire Wire Line
@@
 Connection ~ 15950 9750
 Connection ~ 15950 9900
-Connection ~ 15950 10050
-Connection ~ 15950 10200
 Connection ~ 15950 10350
 Connection ~ 16250 7100
@@
 Connection ~ 15750 9750
 Connection ~ 15750 9900
-Connection ~ 15750 10050
-Connection ~ 15750 10200
 Connection ~ 15750 10350
 Connection ~ 16050 7200
@@
 Wire Notes Line
 	21550 10800 21550 11300
+Wire Wire Line
+	15750 10200 15750 10350
+Connection ~ 15750 10200
+Wire Wire Line
+	15950 10350 15950 10200
+Connection ~ 15950 10200
+$Comp
+L Device:C_Small C67
+U 1 1 617DD991
+P 15850 10200
+F 0 "C67" H 15942 10246 50  0000 L CNN
+F 1 "0.1u" H 15942 10155 50  0000 L CNN
+F 2 "Capacitor_Tantalum_SMD:CP_EIA-2012-15_AVX-P" H 15850 10200 50  0001 C CNN
+F 3 "~" H 15850 10200 50  0001 C CNN
+	1    15850 10200
+	0    1    1    0
+$EndComp
+Wire Wire Line
+	15950 9900 15950 10200
+Wire Wire Line
+	15750 9900 15750 10200
 $EndSCHEMATC

Commit message: removed mounting holes
Parts:
- removed H1: MountingHole_Pad, acheron_MountingHoles:MoutingHole_Oval_7mm_5.0x2.5mm, symbol Mechanical:MountingHole_Pad
- removed H10, H2, H5, H6, H7, H8, H9: MountingHole, acheron_MountingHoles:MoutingHole_Oval_7mm_5.0x2.5mm, symbol Mechanical:MountingHole
- removed H3, H4: MountingHole, acheron_MountingHoles:halfSideHole, symbol Mechanical:MountingHole
Connections:
- net labels removed: CASE
Other:
- note removed: "Mounting Holes"
Changed lines of the file:
@@
 $EndComp
 $Comp
-L Mechanical:MountingHole_Pad H1
-U 1 1 63E6633A
-P 20200 7850
-F 0 "H1" V 20154 8000 50  0000 L CNN
-F 1 "MountingHole_Pad" V 20245 8000 50  0000 L CNN
-F 2 "acheron_MountingHoles:MoutingHole_Oval_7mm_5.0x2.5mm" H 20200 7850 50  0001 C CNN
-F 3 "~" H 20200 7850 50  0001 C CNN
-	1    20200 7850
-	0    1    1    0
-$EndComp
-$Comp
-L Mechanical:MountingHole H2
-U 1 1 63E695B6
-P 20250 8050
-F 0 "H2" H 20350 8096 50  0000 L CNN
-F 1 "MountingHole" H 20350 8005 50  0000 L CNN
-F 2 "acheron_MountingHoles:MoutingHole_Oval_7mm_5.0x2.5mm" H 20250 8050 50  0001 C CNN
-F 3 "~" H 20250 8050 50  0001 C CNN
-	1    20250 8050
-	1    0    0    -1
-$EndComp
-$Comp
-L Mechanical:MountingHole H3
-U 1 1 63E6C1F7
-P 20250 8250
-F 0 "H3" H 20350 8296 50  0000 L CNN
-F 1 "MountingHole" H 20350 8205 50  0000 L CNN
-F 2 "acheron_MountingHoles:halfSideHole" H 20250 8250 50  0001 C CNN
-F 3 "~" H 20250 8250 50  0001 C CNN
-	1    20250 8250
-	1    0    0    -1
-$EndComp
-$Comp
-L Mechanical:MountingHole H4
-U 1 1 63F0BE48
-P 20250 8450
-F 0 "H4" H 20350 8496 50  0000 L CNN
-F 1 "MountingHole" H 20350 8405 50  0000 L CNN
-F 2 "acheron_MountingHoles:halfSideHole" H 20250 8450 50  0001 C CNN
-F 3 "~" H 20250 8450 50  0001 C CNN
-	1    20250 8450
-	1    0    0    -1
-$EndComp
-$Comp
-L Mechanical:MountingHole H5
-U 1 1 63FABAC8
-P 20250 8650
-F 0 "H5" H 20350 8696 50  0000 L CNN
-F 1 "MountingHole" H 20350 8605 50  0000 L CNN
-F 2 "acheron_MountingHoles:MoutingHole_Oval_7mm_5.0x2.5mm" H 20250 8650 50  0001 C CNN
-F 3 "~" H 20250 8650 50  0001 C CNN
-	1    20250 8650
-	1    0    0    -1
-$EndComp
-$Comp
-L Mechanical:MountingHole H6
-U 1 1 6404B7A4
-P 20250 8850
-F 0 "H6" H 20350 8896 50  0000 L CNN
-F 1 "MountingHole" H 20350 8805 50  0000 L CNN
-F 2 "acheron_MountingHoles:MoutingHole_Oval_7mm_5.0x2.5mm" H 20250 8850 50  0001 C CNN
-F 3 "~" H 20250 8850 50  0001 C CNN
-	1    20250 8850
-	1    0    0    -1
-$EndComp
-$Comp
-L Mechanical:MountingHole H7
-U 1 1 640EB3BA
-P 20250 9050
-F 0 "H7" H 20350 9096 50  0000 L CNN
-F 1 "MountingHole" H 20350 9005 50  0000 L CNN
-F 2 "acheron_MountingHoles:MoutingHole_Oval_7mm_5.0x2.5mm" H 20250 9050 50  0001 C CNN
-F 3 "~" H 20250 9050 50  0001 C CNN
-	1    20250 9050
-	1    0    0    -1
-$EndComp
-$Comp
-L Mechanical:MountingHole H8
-U 1 1 6418B100
-P 20250 9250
-F 0 "H8" H 20350 9296 50  0000 L CNN
-F 1 "MountingHole" H 20350 9205 50  0000 L CNN
-F 2 "acheron_MountingHoles:MoutingHole_Oval_7mm_5.0x2.5mm" H 20250 9250 50  0001 C CNN
-F 3 "~" H 20250 9250 50  0001 C CNN
-	1    20250 9250
-	1    0    0    -1
-$EndComp
-$Comp
-L Mechanical:MountingHole H9
-U 1 1 6422AC47
-P 20250 9450
-F 0 "H9" H 20350 9496 50  0000 L CNN
-F 1 "MountingHole" H 20350 9405 50  0000 L CNN
-F 2 "acheron_MountingHoles:MoutingHole_Oval_7mm_5.0x2.5mm" H 20250 9450 50  0001 C CNN
-F 3 "~" H 20250 9450 50  0001 C CNN
-	1    20250 9450
-	1    0    0    -1
-$EndComp
-$Comp
-L Mechanical:MountingHole H10
-U 1 1 642CA7E6
-P 20250 9650
-F 0 "H10" H 20350 9696 50  0000 L CNN
-F 1 "MountingHole" H 20350 9605 50  0000 L CNN
-F 2 "acheron_MountingHoles:MoutingHole_Oval_7mm_5.0x2.5mm" H 20250 9650 50  0001 C CNN
-F 3 "~" H 20250 9650 50  0001 C CNN
-	1    20250 9650
-	1    0    0    -1
-$EndComp
-$Comp
 L Diode:1N914 D3
 U 1 1 644B8699
@@
 Text GLabel 23650 13350 2    50   BiDi ~ 0
 DBUS+
-Text GLabel 20100 7850 0    50   Input ~ 0
-CASE
 Text GLabel 22400 11700 0    50   Input ~ 0
 Case
@@
 Text Notes 22100 11450 0    50   ~ 0
 Case ESD
-Text Notes 19900 7750 0    50   ~ 0
-Mounting Holes
 Text Notes 22100 12550 0    50   ~ 0
 USB ESD Protection
@@
 	22050 14250 22050 12450
 Wire Notes Line
-	19850 7650 19850 9800
-Wire Notes Line
-	19850 9800 21050 9800
-Wire Notes Line
-	21050 9800 21050 7650
-Wire Notes Line
-	21050 7650 19850 7650
-Wire Notes Line
 	19850 14250 21950 14250
 Wire Notes Line
@@
 Wire Wire Line
 	15750 9900 15750 10200
+Entry Wire Line
+	19150 12250 19250 12350
 $EndSCHEMATC

Commit message: added 3d models
3d models for components and pcb
plate svg n stuff
Parts:
- LED1, LED10, LED11, LED12, LED13, LED14, LED15, LED16, LED17, LED18, LED19, LED2, LED20, LED21, LED22, LED23, LED24, LED25, LED26, LED27, LED28, LED29, LED3, LED30, LED31, LED32, LED33, LED34, LED35, LED36, LED37, LED38, LED39, LED4, LED40, LED41, LED42, LED43, LED44, LED45, LED46, LED47, LED48, LED49, LED5, LED50, LED51, LED52, LED53, LED54, LED55, LED56, LED57, LED58, LED59, LED6, LED60, LED61, LED62, LED63, LED64, LED65, LED66, LED67, LED68, LED69, LED7, LED70, LED71, LED72, LED73, LED74, LED75, LED76, LED77, LED78, LED79, LED8, LED80, LED81, LED82, LED83, LED84, LED85, LED86, LED9: footprint WS2812B:WS2812B -> WS2812B:LED_SK6812MINI_PLCC4_3.5x3.5mm_P1.75mm; symbol ws2812b:WS2812B -> ws2812b:SK6812MINI_V2
Connections:
- net 5V_1000u: now also LED1.4 (VCC), LED10.4 (VCC), LED11.4 (VCC), LED12.4 (VCC), LED13.4 (VCC), LED14.4 (VCC), LED15.4 (VCC), LED16.4 (VCC), LED17.4 (VCC), LED18.4 (VCC), LED19.4 (VCC), LED2.4 (VCC), LED20.4 (VCC), LED21.4 (VCC), LED22.4 (VCC), LED23.4 (VCC), LED24.4 (VCC), LED25.4 (VCC), LED26.4 (VCC), LED27.4 (VCC), LED28.4 (VCC), LED29.4 (VCC), LED3.4 (VCC), LED30.4 (VCC), LED31.4 (VCC), LED32.4 (VCC), LED33.4 (VCC), LED34.4 (VCC), LED35.4 (VCC), LED36.4 (VCC), LED37.4 (VCC), LED38.4 (VCC), LED39.4 (VCC), LED4.4 (VCC), LED40.4 (VCC), LED41.4 (VCC), LED42.4 (VCC), LED43.4 (VCC), LED44.4 (VCC), LED45.4 (VCC), LED46.4 (VCC), LED47.4 (VCC), LED48.4 (VCC), LED49.4 (VCC), LED5.4 (VCC), LED50.4 (VCC), LED51.4 (VCC), LED52.4 (VCC), LED53.4 (VCC), LED54.4 (VCC), LED55.4 (VCC), LED56.4 (VCC), LED57.4 (VCC), LED58.4 (VCC), LED59.4 (VCC), LED6.4 (VCC), LED60.4 (VCC), LED61.4 (VCC), LED62.4 (VCC), LED63.4 (VCC), LED64.4 (VCC), LED65.4 (VCC), LED66.4 (VCC), LED67.4 (VCC), LED68.4 (VCC), LED69.4 (VCC), LED7.4 (VCC), LED70.4 (VCC), LED71.4 (VCC), LED72.4 (VCC), LED73.4 (VCC), LED74.4 (VCC), LED75.4 (VCC), LED76.4 (VCC), LED77.4 (VCC), LED78.4 (VCC), LED79.4 (VCC), LED8.4 (VCC), LED80.4 (VCC), LED81.4 (VCC), LED82.4 (VCC), LED83.4 (VCC), LED84.4 (VCC), LED85.4 (VCC), LED86.4 (VCC), LED9.4 (VCC); no longer LED1.1 (VCC), LED10.1 (VCC), LED11.1 (VCC), LED12.1 (VCC), LED13.1 (VCC), LED14.1 (VCC), LED15.1 (VCC), LED16.1 (VCC), LED17.1 (VCC), LED18.1 (VCC), LED19.1 (VCC), LED2.1 (VCC), LED20.1 (VCC), LED21.1 (VCC), LED22.1 (VCC), LED23.1 (VCC), LED24.1 (VCC), LED25.1 (VCC), LED26.1 (VCC), LED27.1 (VCC), LED28.1 (VCC), LED29.1 (VCC), LED3.1 (VCC), LED30.1 (VCC), LED31.1 (VCC), LED32.1 (VCC), LED33.1 (VCC), LED34.1 (VCC), LED35.1 (VCC), LED36.1 (VCC), LED37.1 (VCC), LED38.1 (VCC), LED39.1 (VCC), LED4.1 (VCC), LED40.1 (VCC), LED41.1 (VCC), LED42.1 (VCC), LED43.1 (VCC), LED44.1 (VCC), LED45.1 (VCC), LED46.1 (VCC), LED47.1 (VCC), LED48.1 (VCC), LED49.1 (VCC), LED5.1 (VCC), LED50.1 (VCC), LED51.1 (VCC), LED52.1 (VCC), LED53.1 (VCC), LED54.1 (VCC), LED55.1 (VCC), LED56.1 (VCC), LED57.1 (VCC), LED58.1 (VCC), LED59.1 (VCC), LED6.1 (VCC), LED60.1 (VCC), LED61.1 (VCC), LED62.1 (VCC), LED63.1 (VCC), LED64.1 (VCC), LED65.1 (VCC), LED66.1 (VCC), LED67.1 (VCC), LED68.1 (VCC), LED69.1 (VCC), LED7.1 (VCC), LED70.1 (VCC), LED71.1 (VCC), LED72.1 (VCC), LED73.1 (VCC), LED74.1 (VCC), LED75.1 (VCC), LED76.1 (VCC), LED77.1 (VCC), LED78.1 (VCC), LED79.1 (VCC), LED8.1 (VCC), LED80.1 (VCC), LED81.1 (VCC), LED82.1 (VCC), LED83.1 (VCC), LED84.1 (VCC), LED85.1 (VCC), LED86.1 (VCC), LED9.1 (VCC)
- net GND: now also LED1.2 (GND), LED10.2 (GND), LED11.2 (GND), LED12.2 (GND), LED13.2 (GND), LED14.2 (GND), LED15.2 (GND), LED16.2 (GND), LED17.2 (GND), LED18.2 (GND), LED19.2 (GND), LED2.2 (GND), LED20.2 (GND), LED21.2 (GND), LED22.2 (GND), LED23.2 (GND), LED24.2 (GND), LED25.2 (GND), LED26.2 (GND), LED27.2 (GND), LED28.2 (GND), LED29.2 (GND), LED3.2 (GND), LED30.2 (GND), LED31.2 (GND), LED32.2 (GND), LED33.2 (GND), LED34.2 (GND), LED35.2 (GND), LED36.2 (GND), LED37.2 (GND), LED38.2 (GND), LED39.2 (GND), LED4.2 (GND), LED40.2 (GND), LED41.2 (GND), LED42.2 (GND), LED43.2 (GND), LED44.2 (GND), LED45.2 (GND), LED46.2 (GND), LED47.2 (GND), LED48.2 (GND), LED49.2 (GND), LED5.2 (GND), LED50.2 (GND), LED51.2 (GND), LED52.2 (GND), LED53.2 (GND), LED54.2 (GND), LED55.2 (GND), LED56.2 (GND), LED57.2 (GND), LED58.2 (GND), LED59.2 (GND), LED6.2 (GND), LED60.2 (GND), LED61.2 (GND), LED62.2 (GND), LED63.2 (GND), LED64.2 (GND), LED65.2 (GND), LED66.2 (GND), LED67.2 (GND), LED68.2 (GND), LED69.2 (GND), LED7.2 (GND), LED70.2 (GND), LED71.2 (GND), LED72.2 (GND), LED73.2 (GND), LED74.2 (GND), LED75.2 (GND), LED76.2 (GND), LED77.2 (GND), LED78.2 (GND), LED79.2 (GND), LED8.2 (GND), LED80.2 (GND), LED81.2 (GND), LED82.2 (GND), LED83.2 (GND), LED84.2 (GND), LED85.2 (GND), LED86.2 (GND), LED9.2 (GND); no longer LED1.3 (GND), LED10.3 (GND), LED11.3 (GND), LED12.3 (GND), LED13.3 (GND), LED14.3 (GND), LED15.3 (GND), LED16.3 (GND), LED17.3 (GND), LED18.3 (GND), LED19.3 (GND), LED2.3 (GND), LED20.3 (GND), LED21.3 (GND), LED22.3 (GND), LED23.3 (GND), LED24.3 (GND), LED25.3 (GND), LED26.3 (GND), LED27.3 (GND), LED28.3 (GND), LED29.3 (GND), LED3.3 (GND), LED30.3 (GND), LED31.3 (GND), LED32.3 (GND), LED33.3 (GND), LED34.3 (GND), LED35.3 (GND), LED36.3 (GND), LED37.3 (GND), LED38.3 (GND), LED39.3 (GND), LED4.3 (GND), LED40.3 (GND), LED41.3 (GND), LED42.3 (GND), LED43.3 (GND), LED44.3 (GND), LED45.3 (GND), LED46.3 (GND), LED47.3 (GND), LED48.3 (GND), LED49.3 (GND), LED5.3 (GND), LED50.3 (GND), LED51.3 (GND), LED52.3 (GND), LED53.3 (GND), LED54.3 (GND), LED55.3 (GND), LED56.3 (GND), LED57.3 (GND), LED58.3 (GND), LED59.3 (GND), LED6.3 (GND), LED60.3 (GND), LED61.3 (GND), LED62.3 (GND), LED63.3 (GND), LED64.3 (GND), LED65.3 (GND), LED66.3 (GND), LED67.3 (GND), LED68.3 (GND), LED69.3 (GND), LED7.3 (GND), LED70.3 (GND), LED71.3 (GND), LED72.3 (GND), LED73.3 (GND), LED74.3 (GND), LED75.3 (GND), LED76.3 (GND), LED77.3 (GND), LED78.3 (GND), LED79.3 (GND), LED8.3 (GND), LED80.3 (GND), LED81.3 (GND), LED82.3 (GND), LED83.3 (GND), LED84.3 (GND), LED85.3 (GND), LED86.3 (GND), LED9.3 (GND)
- net at R4.2: now also LED84.3 (DIN); no longer LED84.4 (DIN)
- new net: LED72.3 (DIN), LED83.1 (DOUT)
- new net: LED83.3 (DIN), LED86.1 (DOUT)
- new net: LED1.1 (DOUT), LED85.3 (DIN)
- new net: LED1.3 (DIN), LED7.1 (DOUT)
- new net: LED13.1 (DOUT), LED7.3 (DIN)
- new net: LED13.3 (DIN), LED19.1 (DOUT)
- new net: LED19.3 (DIN), LED25.1 (DOUT)
- new net: LED25.3 (DIN), LED31.1 (DOUT)
- new net: LED31.3 (DIN), LED37.1 (DOUT)
- new net: LED37.3 (DIN), LED43.1 (DOUT)
- new net: LED43.3 (DIN), LED49.1 (DOUT)
- new net: LED49.3 (DIN), LED55.1 (DOUT)
- new net: LED55.3 (DIN), LED61.1 (DOUT)
- new net: LED61.3 (DIN), LED67.1 (DOUT)
- new net: LED67.3 (DIN), LED73.1 (DOUT)
- new net: LED73.3 (DIN), LED84.1 (DOUT)
- new net: LED2.1 (DOUT), LED82.3 (DIN)
- new net: LED2.3 (DIN), LED8.1 (DOUT)
- new net: LED14.1 (DOUT), LED8.3 (DIN)
- new net: LED14.3 (DIN), LED20.1 (DOUT)
- new net: LED20.3 (DIN), LED26.1 (DOUT)
- new net: LED26.3 (DIN), LED32.1 (DOUT)
- new net: LED32.3 (DIN), LED38.1 (DOUT)
- new net: LED38.3 (DIN), LED44.1 (DOUT)
- new net: LED44.3 (DIN), LED50.1 (DOUT)
- new net: LED50.3 (DIN), LED56.1 (DOUT)
- new net: LED56.3 (DIN), LED62.1 (DOUT)
- new net: LED62.3 (DIN), LED68.1 (DOUT)
- new net: LED68.3 (DIN), LED74.1 (DOUT)
- new net: LED74.3 (DIN), LED78.1 (DOUT)
- new net: LED3.1 (DOUT), LED80.3 (DIN)
- new net: LED3.3 (DIN), LED9.1 (DOUT)
- new net: LED15.1 (DOUT), LED9.3 (DIN)
- new net: LED15.3 (DIN), LED21.1 (DOUT)
- new net: LED21.3 (DIN), LED27.1 (DOUT)
- new net: LED27.3 (DIN), LED33.1 (DOUT)
- new net: LED33.3 (DIN), LED39.1 (DOUT)
- new net: LED39.3 (DIN), LED45.1 (DOUT)
- new net: LED45.3 (DIN), LED51.1 (DOUT)
- new net: LED51.3 (DIN), LED57.1 (DOUT)
- new net: LED57.3 (DIN), LED63.1 (DOUT)
- new net: LED63.3 (DIN), LED69.1 (DOUT)
- new net: LED69.3 (DIN), LED75.1 (DOUT)
- new net: LED75.3 (DIN), LED79.1 (DOUT)
- new net: LED4.1 (DOUT), LED81.3 (DIN)
- new net: LED10.1 (DOUT), LED4.3 (DIN)
- new net: LED10.3 (DIN), LED16.1 (DOUT)
- new net: LED16.3 (DIN), LED22.1 (DOUT)
- new net: LED22.3 (DIN), LED28.1 (DOUT)
- new net: LED28.3 (DIN), LED34.1 (DOUT)
- new net: LED34.3 (DIN), LED40.1 (DOUT)
- new net: LED40.3 (DIN), LED46.1 (DOUT)
- new net: LED46.3 (DIN), LED52.1 (DOUT)
- new net: LED52.3 (DIN), LED58.1 (DOUT)
- new net: LED58.3 (DIN), LED64.1 (DOUT)
- new net: LED64.3 (DIN), LED70.1 (DOUT)
- new net: LED70.3 (DIN), LED76.1 (DOUT)
- new net: LED76.3 (DIN), LED80.1 (DOUT)
- new net: LED5.1 (DOUT), LED86.3 (DIN)
- new net: LED11.1 (DOUT), LED5.3 (DIN)
- new net: LED11.3 (DIN), LED17.1 (DOUT)
- new net: LED17.3 (DIN), LED23.1 (DOUT)
- new net: LED23.3 (DIN), LED29.1 (DOUT)
- new net: LED29.3 (DIN), LED35.1 (DOUT)
- new net: LED35.3 (DIN), LED41.1 (DOUT)
- new net: LED41.3 (DIN), LED47.1 (DOUT)
- new net: LED47.3 (DIN), LED53.1 (DOUT)
- new net: LED53.3 (DIN), LED59.1 (DOUT)
- new net: LED59.3 (DIN), LED65.1 (DOUT)
- new net: LED65.3 (DIN), LED71.1 (DOUT)
- new net: LED71.3 (DIN), LED77.1 (DOUT)
- new net: LED77.3 (DIN), LED81.1 (DOUT)
- new net: LED78.3 (DIN), LED85.1 (DOUT)
- new net: LED79.3 (DIN), LED82.1 (DOUT)
- new net: LED12.1 (DOUT), LED6.3 (DIN)
- new net: LED12.3 (DIN), LED18.1 (DOUT)
- new net: LED18.3 (DIN), LED24.1 (DOUT)
- new net: LED24.3 (DIN), LED30.1 (DOUT)
- new net: LED30.3 (DIN), LED36.1 (DOUT)
- new net: LED36.3 (DIN), LED42.1 (DOUT)
- new net: LED42.3 (DIN), LED48.1 (DOUT)
- new net: LED48.3 (DIN), LED54.1 (DOUT)
- new net: LED54.3 (DIN), LED60.1 (DOUT)
- new net: LED60.3 (DIN), LED66.1 (DOUT)
- new net: LED66.3 (DIN), LED72.1 (DOUT)

Commit message: bruh moment
Connections:
- net col1: now also MX54.1 (COL), MX71.1 (COL); no longer MX5.1 (COL), MX6.1 (COL)
- net col5: no longer MX54.1 (COL)
- net col6: no longer MX71.1 (COL)
- net col7: now also MX5.1 (COL), MX6.1 (COL)
Changed lines of the file:
@@
 	25650 8500 25650 9250
 Wire Wire Line
-	25650 9250 25650 10000
-Wire Wire Line
-	25650 10000 25650 10750
-Wire Wire Line
 	26000 10750 26000 10000
 Wire Wire Line
@@
 	29500 9250 29500 8500
 Wire Wire Line
-	29500 10000 29500 9250
-Wire Wire Line
 	29150 6850 29150 7000
 Wire Wire Line
@@
 	24000 7550 24100 7550
 Wire Wire Line
-	29500 10000 29500 10750
-Wire Wire Line
 	29150 10750 29150 10000
 Wire Wire Line
 	28800 10000 28800 10750
-Wire Wire Line
-	28450 10750 28450 10000
 Wire Wire Line
 	28100 10000 28100 10750
@@
 Connection ~ 25650 7750
 Connection ~ 25650 8500
-Connection ~ 25650 9250
-Connection ~ 25650 10000
 Connection ~ 26000 7000
 Connection ~ 26000 7750
@@
 Connection ~ 28450 8500
 Connection ~ 28450 9250
-Connection ~ 28450 10000
 Connection ~ 28800 7000
 Connection ~ 28800 7750
@@
 Connection ~ 29500 7750
 Connection ~ 29500 8500
-Connection ~ 29500 9250
 Connection ~ 29150 6850
 Connection ~ 25450 7550
@@
 Text GLabel 17650 10850 0    50   Input ~ 0
 E_CCW2
-Connection ~ 29500 10000
 Wire Wire Line
 	29300 11250 29300 11350
@@
 Entry Wire Line
 	19150 12250 19250 12350
+Wire Wire Line
+	25650 10000 25650 10750
+Wire Wire Line
+	29150 10750 29500 10750
+Connection ~ 29150 10750
+Text GLabel 25650 10200 2    50   Input ~ 0
+col7
+Text GLabel 29500 10000 1    50   Input ~ 0
+col1
+Text GLabel 28450 10750 1    50   Input ~ 0
+col1
 $EndSCHEMATC
