File: Peripherals/macro-numpad/numpad.sch (KiCad schematic (older format))
At the start: 40 parts

Commit message: bruh moment
Parts:
- added C? (x4): 100n, Capacitor_Tantalum_SMD:CP_EIA-2012-15_AVX-P, symbol Device:C
- added C? (x2): 4.7u, Capacitor_Tantalum_SMD:CP_EIA-2012-15_AVX-P, symbol Device:C
- added C?: 10n, Capacitor_Tantalum_SMD:CP_EIA-2012-15_AVX-P, symbol Device:C
- added C?: 1u, Capacitor_Tantalum_SMD:CP_EIA-2012-15_AVX-P, symbol Device:C
- added C? (x2): 4.7n, Capacitor_Tantalum_SMD:CP_EIA-2012-15_AVX-P, symbol Device:C_Small
- added C? (x4): 100n, Capacitor_Tantalum_SMD:CP_EIA-2012-15_AVX-P, symbol Device:C_Small
- added D?: B260, Diode_SMD:D_SMB, symbol Diode:B260
- added D? (x2): 1N914, Diode_THT:D_DO-35_SOD27_P7.62mm_Horizontal, symbol Diode:1N914
- added E?: Rotary_Encoder_Switch_Chassis, acheron_Hardware:ALPS_EC11E, symbol acheronSymbols:Rotary_Encoder_Switch_Chassis
- added F?: Polyfuse_Small, Fuse:Fuse_1206_3216Metric, symbol Device:Polyfuse_Small
- added J?: Conn_ARM_JTAG_SWD_10, Connector_PinSocket_1.00mm:PinSocket_2x05_P1.00mm_Vertical_SMD, symbol Connector:Conn_ARM_JTAG_SWD_10
- added JIN?: USB_C_Receptacle_USB2.0, Type-C:USB_C_GCT_USB4085, symbol Connector:USB_C_Receptacle_USB2.0
- added LED? (x2): LED, LED_SMD:LED_0805_2012Metric, symbol Device:LED
- added R? (x2): 5.1k, Resistor_SMD:R_0805_2012Metric, symbol Device:R_Small
- added R?: 22k, Resistor_SMD:R_0805_2012Metric, symbol Device:R_Small
- added R? (x2): 68, Resistor_SMD:R_0805_2012Metric, symbol Device:R
- added R?: 1M, Resistor_SMD:R_0805_2012Metric, symbol Device:R_Small
- added U?: STM32F072CBTx, Package_QFP:LQFP-48_7x7mm_P0.5mm, symbol MCU_ST_STM32F0:STM32F072CBTx
- added U?: MCP1700-3302E_SOT23, Package_TO_SOT_SMD:SOT-23, symbol Regulator_Linear:MCP1700-3302E_SOT23
- added U?: USBLC6-2SC6, Package_TO_SOT_SMD:SOT-23-6, symbol Installation-01-rescue:USBLC6-2SC6-Power_Protection
Connections:
- net labels added: BOOT0, Case, D+, D-, DBUS+, DBUS-, E_Button, E_Button2, E_CCW, E_CCW2, E_CW, E_CW2, GND, IndicatorLED, Keeb_3.3V, Keeb_5V, NRST, RGB_LED, SWCLK, SWDIO, VBUS, VDD, VDDA, VDDIO2, col1, col2, col3, col4, col5, col6, col7, col8, numLockLED, row1, row10, row11, row12, row2, row3, row4, row5, row6, row7, row8, row9
- wire segments 40 -> 184
- no-connect marks 0 -> 8
Other:
- note added: "ARM CORTEX IC"
- note added: "Case ESD"
- note added: "Indicator LED"
- note added: "Keeb ARM Chip Decoupling Caps"
- note added: "Keeb Power Supply"
- note added: "Num Lock LED"
- note added: "Rotary Encoder"
- note added: "Serial Programmer"
- note added: "USB C IN"
- note added: "USB ESD Protection"
- moved on the sheet: D?, MX?
